File: boards/freesample/psu.sch (KiCad schematic (older format))
At the start: 36 parts, among them U26 MCP1755ST-5002E/MC, U27 LM27761, U28 ADP1763, U29 ADP1763, U30 TPS62130RGTR

Commit message: Continued work on PSU design
Parts:
- added C239, C244, C245: 10 nF, symbol device:C
- added C240, C243: 22 uF 16V, symbol device:C
- added C241, C242, C246, C247, C248, C249: 4.7 uF, symbol device:C
- added R40: FIXME, symbol device:R
- added R41: 1.33K, symbol device:R
- added R42: 20K, symbol device:R
- added R43, R47, R49, R50: 0, symbol device:R
- added R44, R51, R52: 113K, symbol device:R
- added R45, R53, R54: 100K, symbol device:R
- added R46: 10K, symbol device:R
- added R48, R55, R56: 20K 0.1%, symbol device:R
- added U31, U33, U34: ADP1741, symbol power-azonenberg:ADP1741
- added U32: OKL-T/3-W12P-C, symbol power-azonenberg:OLK-T_3-W12P-C
Connections:
- net 12V0: now also C240.1, R42.2, U32.2 (VIN)
- net 3V3: now also C249.2, R50.2, U34.10 (VOUT), U34.11 (VOUT), U34.12 (VOUT), U34.13 (VOUT), U34.14 (VOUT)
- net 5V0: now also C243.1, R47.1, U32.4 (VOUT)
- net D3V3: now also R45.1, R46.1, R53.1, R54.1
- net GND: now also C239.2, C240.2, C241.2, C242.1, C243.2, C244.2, C245.2, C246.2, C247.2, C248.1, C249.1, R40.2, R41.1, R48.1, R55.1, R56.1, U31.6 (GND), U31.PAD (GND), U32.3 (GND), U32.7 (GND), U33.6 (GND), U33.PAD (GND), U34.6 (GND), U34.PAD (GND)
- net 1V0_VADJ: now reaches U28.8 (VADJ)
- net 1V0_VADJ: now also U29.8 (VADJ), R40.1
- net 1V15_PGOOD: now reaches R37.1, U30.4 (PG)
- new net: R42.1, U32.1 (EN)
- new net: R41.2, U32.6 (TRIM)
- new net: C239.1, U31.7 (SS)
- new net: R44.2, R48.2, U31.9 (ADJ)
- new net: C244.1, U33.7 (SS)
- new net: R51.2, R55.2, U33.9 (ADJ)
- new net: C245.1, U34.7 (SS)
- new net: R52.2, R56.2, U34.9 (ADJ)
- new net 3V3_CLKBUF: C242.2, R43.2, U31.10 (VOUT), U31.11 (VOUT), U31.12 (VOUT), U31.13 (VOUT), U31.14 (VOUT)
- new net 3V3_CLKBUF_PGOOD: R45.2, U31.5 (PG)
- new net 3V3_CLKBUF_SENSE: R43.1, R44.1
- new net 3V3_PGOOD: R54.2, U34.5 (PG)
- new net 3V3_PLL: C248.2, R49.2, U33.10 (VOUT), U33.11 (VOUT), U33.12 (VOUT), U33.13 (VOUT), U33.14 (VOUT)
- new net 3V3_PLL_PGOOD: R53.2, U33.5 (PG)
- new net 3V3_PLL_SENSE: R49.1, R51.1
- new net 3V3_SENSE: R50.1, R52.1
- new net 3V5_INT: C241.1, C246.1, C247.1, U31.1 (VIN), U31.15 (VIN), U31.16 (VIN), U31.2 (VIN), U31.3 (VIN), U31.4 (EN), U33.1 (VIN), U33.15 (VIN), U33.16 (VIN), U33.2 (VIN), U33.3 (VIN), U33.4 (EN), U34.1 (VIN), U34.15 (VIN), U34.16 (VIN), U34.2 (VIN), U34.3 (VIN), U34.4 (EN)
- new net 5V0_PGOOD: R46.2, U32.10 (PGOOD)
- new net 5V0_SENSE: R47.2, U32.5 (SENSE)
- no-connect marks 2 -> 1
Other:
- note added: "+3.3V supply for PLL and VCO (0.85A)"
- note added: "+3.3V supply for clock buffers (1.4A)"
- note added: "+3.3V supply for other loads (0.25A)"
- note added: "+3.5V intermediate rail (2.6A)"
- note added: "+5V intermediate rail for INTEGRALSTICK"
- note added: "0.2V drop * 0.25A = 0.05W\n2.1C rise"
- note added: "0.2V drop * 0.85A = 0.17W\n7.14C rise"
- note added: "0.2V drop * 2A = 0.4W\n16.8C rise\n\nVout = 0.5*(1 + R44/R48), R48 < 60 kR\nR44=113K gives 3.325V"
- note added: "Vout = 3.0 * (Radj * 50 uA)\nRadj = 1V/(150 uA) = 6.667 kR\nUse 6.65K for 0.9975V\n\nConnect two in parallel to spread out heat generation\n0.15V * 3A = 0.45W total, estimate 0.3W worst case per chip\nAssuming 1cm^2 plane for heatsinking, 30.8C rise.\nBigger planes will improve this\nTypical SERDES power is << 3A which will also help,\nespecially if we power down the unused channel"
- note removed: "Connect two in parallel to spread out heat generation\n0.15V * 3A = 0.45W total, estimate 0.3W worst case per chip\nAssuming 1cm^2 plane for heatsinking, 30.8C rise.\nBigger planes will improve this\nTypical SERDES power is << 3A which will also help,\nespecially if we power down the unused channel"

Commit message: Continued PSU design
Parts:
- removed L1: SRP4020TA-2R2M, symbol passive-azonenberg:INDUCTOR_PWROUT
- removed U30: TPS62130RGTR, symbol power-azonenberg:TPS62130RGTR
- added C250, C251, C252, C255: 22 uF 16V, symbol device:C
- added C253, C254, C258, C259: 4.7 uF 5V, symbol device:C
- added C256, C260: 2.2 uF 5V, symbol device:C
- added C257, C261: 1 uF 5V, symbol device:C
- added R57, R61, R65, R71: 0, symbol device:R
- added R58, R62: 2.05K, symbol device:R
- added R59, R63, R69: 20K, symbol device:R
- added R60, R64, R70: 10K, symbol device:R
- added R66, R72: 309K 1%, symbol device:R
- added R67, R73: 100K 1%, symbol device:R
- added R68: 2.8L, symbol device:R
- added U30, U35, U36, U38: OKL-T/3-W12P-C, symbol power-azonenberg:OLK-T_3-W12P-C
- added U37, U39: LM27761, symbol power-azonenberg:LM27761
- C235: value 3.3 nF -> 22 uF 16V
- C236: value 0.1 uF 16V -> 22 uF 16V
- C238: value 22 uF -> 22 uF 16V
- R37: value 10K -> 10.5K
- R38: value 43.2K -> 20K
- R39: value 100K -> 10K
- R41: value 1.33K -> 1.27K
Connections:
- net 1V15_PGOOD is gone; now on net GND: R37.1
- net 12V0: now also C235.1, R38.2, C250.1, C252.1, R59.2, R63.2, R69.2, U30.2 (VIN), U35.2 (VIN), U36.2 (VIN), U38.2 (VIN); no longer C236.2
- net 1V15_INT: now also C236.1, R57.1, U30.4 (VOUT); no longer C238.2, R38.1
- net 3V0_N: now also C256.2, U37.4 (VOUT)
- net 3V3_N: now also C260.2, U39.4 (VOUT)
- net 3V5_INT: no longer C241.1, C246.1, C247.1, U31.1 (VIN), U31.15 (VIN), U31.16 (VIN), U31.2 (VIN), U31.3 (VIN), U33.1 (VIN), U33.15 (VIN), U33.16 (VIN), U33.2 (VIN), U33.3 (VIN), U34.1 (VIN), U34.15 (VIN), U34.16 (VIN), U34.2 (VIN), U34.3 (VIN)
- net 5V0: no longer C243.1, R47.1, U32.4 (VOUT)
- net 5V0_N: now also R66.1, R72.1
- net A5V0: no longer C221.1, U27.1 (VIN), U27.6 (EN)
- net D3V3: now also R39.1, R60.1, R64.1, R70.1; no longer R37.2
- net GND: now also C236.2, C238.2, C250.2, C251.2, C252.2, C253.2, C254.1, C255.2, C256.1, C258.2, C259.1, C260.1, R58.1, R62.1, R67.1, R68.1, R73.1, U30.3 (GND), U30.7 (GND), U35.3 (GND), U35.7 (GND), U36.3 (GND), U36.7 (GND), U37.2 (GND), U37.PAD (GND), U38.3 (GND), U38.7 (GND), U39.2 (GND), U39.PAD (GND); no longer C236.1, C238.1, R39.1
- net 1V15_FB renamed 1V1_PGOOD
- net 1V1_PGOOD: now also U30.10 (PGOOD); no longer R38.2
- new net: R58.2, U35.6 (TRIM)
- new net: R59.1, U35.1 (EN)
- new net: R37.2, U30.6 (TRIM)
- new net: R38.1, U30.1 (EN)
- new net: R68.2, U38.6 (TRIM)
- new net: R69.1, U38.1 (EN)
- new net: R62.2, U36.6 (TRIM)
- new net: R63.1, U36.1 (EN)
- new net: C254.2, U37.3 (CPOUT)
- new net: C257.1, U37.7 (C1-)
- new net: C257.2, U37.8 (C1+)
- new net: C259.2, U39.3 (CPOUT)
- new net: C261.1, U39.7 (C1-)
- new net: C261.2, U39.8 (C1+)
- new net 1V1_SENSE: R57.2, U30.5 (SENSE)
- new net 2V7_INT: C255.1, R71.1, U38.4 (VOUT)
- new net 2V7_PGOOD: R70.2, U38.10 (PGOOD)
- new net 2V7_SENSE: R71.2, U38.5 (SENSE)
- new net 3V0_N_FB: R66.2, R67.2, U37.5 (VFB)
- new net 3V3_N_FB: R72.2, R73.2, U39.5 (VFB)
- new net 3V5_INT1: C238.1, C246.1, C247.1, C253.1, C258.1, R61.1, U33.1 (VIN), U33.15 (VIN), U33.16 (VIN), U33.2 (VIN), U33.3 (VIN), U34.1 (VIN), U34.15 (VIN), U34.16 (VIN), U34.2 (VIN), U34.3 (VIN), U35.4 (VOUT), U37.1 (VIN), U37.6 (EN), U39.1 (VIN), U39.6 (EN)
- new net 3V5_INT2: C241.1, C251.1, R65.1, U31.1 (VIN), U31.15 (VIN), U31.16 (VIN), U31.2 (VIN), U31.3 (VIN), U36.4 (VOUT)
- new net 3V5_PGOOD: R60.2, U35.10 (PGOOD)
- new net 3V5_PGOOD2: R64.2, U36.10 (PGOOD)
- new net 3V5_SENSE: R61.2, U35.5 (SENSE)
- new net 3V5_SENSE2: R65.2, U36.5 (SENSE)
- new net 5V25: C221.1, C243.1, R47.1, U27.1 (VIN), U27.6 (EN), U32.4 (VOUT)
- no-connect marks 1 -> 5
Other:
- note added: "+1.8V supply for SERDES/comparators (0.2A)"
- note added: "+2.5V supply for flipflops (0.5A)"
- note added: "+2.7V intermediate rail (0.7A)"
- note added: "+3.5V intermediate rail 1 (1.4A)"
- note added: "+3.5V intermediate rail 2 (1.4A)"
- note added: "+5.25V supply for INTEGRALSTICK (<1A typ)"
- note added: "+5V analog supply (<10 mA)"
- note added: "-3.0V supply for comparators (0.1A)"
- note added: "-3.3V supply for delay line (0.2A)"
- note added: "-5V analog supply (3 mA)"
- note added: "1.0V CDR SERDES supply (2.6A)"
- note added: "1.15V intermediate rail (2.6A)"
- note added: "3V0_N: estimated 100 mA from 3.5V in\nVout = -1.22 * (R66+R67)/R67\nR67 > 50 kR (use 100K)\nUse XX (ideal XX) for -3.0V\n\nThermal analysis TODO"
- note added: "3V3_N: estimated 100 mA from 3.5V in\nVout = -1.22 * (R66+R67)/R67\nR67 > 50 kR (use 100K)\nUse XX (ideal XX) for -3.3V\n\nThermal analysis TODO"
- note added: "5V0_N: estimated 3 mA from 5.25V in\nVout = -1.22 * (R28+R29)/R29\nR29 > 50 kR (use 100K\nUse 309K (ideal 309.836K) for -4.99V\n\nSMPS w/ 3 mA load, no thermal\nanalysis necessary"
- note added: "A5V0: estimated 3 mA from 12V in\nConservatively: 4.9C rise (70 mW) at 10 mA"
- note added: "Rtrim(k) = 5.91 / (1.15 - 0.591) = 10.57K nominal"
- note added: "Rtrim(k) = 5.91 / (2.7 - 0.591) = 2.80K nominal"
- note added: "Rtrim(k) = 5.91 / (3.5 - 0.591) = 2.03K nominal"
- note added: "Rtrim(k) = 5.91 / (5.25 - 0.591) = 1.27K"
- note removed: "+3.5V intermediate rail (2.6A)"
- note removed: "+5V analog supply"
- note removed: "+5V intermediate rail for INTEGRALSTICK"
- note removed: "-5V analog supply"
- note removed: "1.0V CDR SERDES supply"
- note removed: "1.15V intermediate rail"
- note removed: "2.5 MHz switching freq\nNormal voltage range\n\nR1 = R2*(Vout/0.8V - 1)\nR2 <= 400K\nR1 = 43.2K, R2 = 100K gives 1.145V"
- note removed: "5V0_N: estimated 3 mA from 5V in\nVout = -1.22 * (R28+R29)/R29\nR29 > 50 kR (use 100K\nUse 309K (ideal 309.836K) for -4.99V\n\nSMPS w/ 3 mA load, no thermal\nanalysis necessary"
- note removed: "A5V0: estimated 3 mA from 12V in\nAdd 1 mA for charge pump and\n3 mA for negative rail = 7 mA\nConservatively: 4.9C rise (70 mW) at 10 mA"
- note removed: "Overall power topology:\n* LDO 12V -> 5V 0.05A for +5V0_A rail\n* Buck 12V -> 5V 5A for intermediate digital rail"
- note removed: "Total power budget (with safety margins included):\n* -5 0.003A\n* -3.3 0.25A\n* -3.0 0.2A\n* +1.0 3A\n* +1.8 0.3A\n* +2.5 0.6A\n* +3.3 3A\n* +5 0.03A\nPlus 5V 1.5A for INTEGRALSTICK"
- moved on the sheet: C225, C226, C227, C228, C229, C230, C231, C232, C233, C234, R30, R31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

Commit message: Lots of ERC fixes, added CML-to-LVDS buffers for FPGA input signals
Connections:
- net 3V5_INT is gone; now on net 3V5_INT1: U31.4 (EN), U33.4 (EN), U34.4 (EN)
- net 5V0 is gone; now on net 1V15_INT: U28.16 (EN), U29.16 (EN)
Changed lines of the file:
@@
 	1000 6800 1700 6800
 Text Label 1700 6900 2    50   ~ 0
-5V0
+1V15_INT
 $Comp
 L device:C C228
@@
 Wire Wire Line
 	1700 8700 1700 8800
-Text Label 1700 8500 2    50   ~ 0
-5V0
 $Comp
 L device:C C232
@@
 $EndComp
 Text Label 5450 3250 2    50   ~ 0
-3V5_INT
+3V5_INT1
 Wire Wire Line
 	5450 3150 4850 3150
@@
 $EndComp
 Text Label 5450 5300 2    50   ~ 0
-3V5_INT
+3V5_INT1
 Wire Wire Line
 	5450 5200 4850 5200
@@
 $EndComp
 Text Label 5500 7250 2    50   ~ 0
-3V5_INT
+3V5_INT1
 Wire Wire Line
 	5500 7150 4900 7150
@@
 	0    1    1    0
 $EndComp
-Text Label 3700 4300 0    50   ~ 0
-D3V3
 Text Label 2900 4300 0    50   ~ 0
 1V1_PGOOD
@@
 Wire Notes Line width 20 style solid
 	8250 4800 12000 4800
+Text HLabel 3700 4300 2    50   Input ~ 0
+D3V3
+Text Label 1700 8500 2    50   ~ 0
+1V15_INT
 $EndSCHEMATC
