File: boards/freesample/oneshot.sch (KiCad schematic (older format))
At the start: 87 parts, among them U18 PI6C59S6005, U19 NB7V52MMNG, U20 NB7V52MMNG, U21 NB7V52MMNG, U22 PI6C59S6005, U23 NB7V52MMNG, U24 PI6C59S6005, U25 SY58051AU, U40 DS25BR150, U7 PI6C59S6005

Commit message: Finished PSU schematic. Ready for design review!
Parts:
- added C313, C314: 0.01 uF, symbol device:C
- added J17, J18: SMA, symbol Connector:Conn_Coaxial
Connections:
- net GND: now also J17.2 (Ext), J18.2 (Ext)
- net CLKOUT_AC_P: now reaches U7.10 (Q4_P)
- net CLKOUT_AC_P: now also C313.2
- net CLKOUT_AC_N: now reaches U7.11 (Q4_N)
- net CLKOUT_AC_N: now also C314.2
- net TRG_P: now reaches U24.1 (Q1_P)
- net TRG_P: now also J17.1 (In)
- net TRG_N: now reaches U24.2 (Q1_N)
- net TRG_N: now also J18.1 (In)
- new net CLKOUT_N: C314.1
- new net CLKOUT_P: C313.1
- no-connect marks 27 -> 23
Changed lines of the file:
@@
 Sheet 6 12
 Title "FREESAMPLE Oscilloscope"
-Date "2019-03-10"
+Date "2019-03-11"
 Rev "0.1"
 Comp "Andrew D. Zonenberg / Antikernel Labs"
@@
 Text Label 4600 6950 0    50   ~ 0
 CLK0_N
-NoConn ~ 3800 8050
-NoConn ~ 3800 8150
 Text Label 2000 3550 2    50   ~ 0
 CLK0_P
@@
 NoConn ~ 14700 2350
 NoConn ~ 14700 2450
-NoConn ~ 14700 2650
-NoConn ~ 14700 2750
 NoConn ~ 14700 2950
 NoConn ~ 14700 3050
@@
 Text Label 1050 9450 2    50   ~ 0
 GND
+Text Label 3800 8050 0    50   ~ 0
+CLKOUT_AC_P
+Text Label 3800 8150 0    50   ~ 0
+CLKOUT_AC_N
+$Comp
+L device:C C?
+U 1 1 5D201188
+P 4350 8050
+AR Path="/5C267736/5D201188" Ref="C?"  Part="1"
+AR Path="/5C15809A/5D201188" Ref="C313"  Part="1"
+F 0 "C313" V 4400 8200 50  0000 C CNN
+F 1 "0.01 uF" V 4300 8250 50  0000 C CNN
+F 2 "" H 4388 7900 50  0001 C CNN
+F 3 "" H 4350 8050 50  0001 C CNN
+	1    4350 8050
+	0    1    -1   0
+$EndComp
+$Comp
+L device:C C?
+U 1 1 5D20195B
+P 4350 8150
+AR Path="/5C267736/5D20195B" Ref="C?"  Part="1"
+AR Path="/5C15809A/5D20195B" Ref="C314"  Part="1"
+F 0 "C314" V 4400 8300 50  0000 C CNN
+F 1 "0.01 uF" V 4300 8350 50  0000 C CNN
+F 2 "" H 4388 8000 50  0001 C CNN
+F 3 "" H 4350 8150 50  0001 C CNN
+	1    4350 8150
+	0    1    -1   0
+$EndComp
+Wire Wire Line
+	3800 8050 4200 8050
+Wire Wire Line
+	4200 8150 3800 8150
+Text HLabel 4750 8050 2    50   Input ~ 0
+CLKOUT_P
+Wire Wire Line
+	4750 8050 4500 8050
+Text HLabel 4750 8150 2    50   Input ~ 0
+CLKOUT_N
+Wire Wire Line
+	4750 8150 4500 8150
+$Comp
+L Connector:Conn_Coaxial J18
+U 1 1 5D291477
+P 15100 2800
+F 0 "J18" H 15200 2775 50  0000 L CNN
+F 1 "SMA" H 15200 2684 50  0000 L CNN
+F 2 "" H 15100 2800 50  0001 C CNN
+F 3 "" H 15100 2800 50  0001 C CNN
+	1    15100 2800
+	1    0    0    -1
+$EndComp
+$Comp
+L Connector:Conn_Coaxial J17
+U 1 1 5D2924E4
+P 15100 2600
+F 0 "J17" H 15200 2482 50  0000 L CNN
+F 1 "SMA" H 15200 2573 50  0000 L CNN
+F 2 "" H 15100 2600 50  0001 C CNN
+F 3 "" H 15100 2600 50  0001 C CNN
+	1    15100 2600
+	1    0    0    1
+$EndComp
+Wire Wire Line
+	14700 2750 14950 2750
+Wire Wire Line
+	14950 2750 14950 2800
+Wire Wire Line
+	14700 2650 14950 2650
+Wire Wire Line
+	14950 2650 14950 2600
+Text Label 15100 2400 0    50   ~ 0
+GND
+Text Label 15100 3000 0    50   ~ 0
+GND
+Text Label 14700 2650 0    50   ~ 0
+TRG_P
+Text Label 14700 2750 0    50   ~ 0
+TRG_N
 $EndSCHEMATC
