File: boards/freesample/oneshot.sch (KiCad schematic (older format))
At the start: 91 parts, among them J17 SMA, J18 SMA, U18 PI6C59S6005, U19 NB7V52MMNG, U20 NB7V52MMNG, U21 NB7V52MMNG, U22 PI6C59S6005, U23 NB7V52MMNG, U24 PI6C59S6005, U25 SY58051AU, U40 DS25BR150, U7 PI6C59S6005

Commit message: Added more test points. Started picking packages for passives. Continued schematic review.
Parts:
- C176, C186, C196, C197, C202, C209: footprint (none) -> azonenberg_pcb:EIA_0603_CAP_NOSILK
- C177, C178, C179, C180, C275, C276, C277, C278, C279, C280, C281, C282, C283, C284, C285, C286, C287, C288, C289, C290, C293, C294, C295, C296, C297, C298, C299, C300, C301, C302, C303, C304, C305, C306, C307, C308, C313, C314: footprint (none) -> azonenberg_pcb:EIA_0201_CAP_NOSILK
- C181, C182, C183, C184, C185, C187, C188, C189, C190, C191, C192, C193, C194, C195, C198, C199, C200, C201, C203, C204, C207, C208, C210, C211, C212, C213, C311: footprint (none) -> azonenberg_pcb:EIA_0402_CAP_NOSILK
- J17, J18: footprint (none) -> azonenberg_pcb:CONN_SMA_EDGE_SAMTEC_SMA_J_P_H_ST_EM1
- JP4, JP5, JP6, JP7: footprint (none) -> azonenberg_pcb:EIA_0402_JUMPER
- R22, R23, R32: footprint (none) -> azonenberg_pcb:EIA_0402_RES_NOSILK
- U18, U22, U24, U7: footprint (none) -> azonenberg_pcb:QFN_24_0.5MM_4x4MM
- U19, U20, U21, U23, U25: footprint (none) -> azonenberg_pcb:QFN_16_0.5MM_3x3MM
- U40: footprint (none) -> azonenberg_pcb:DFN_8_0.5MM_3x3MM

Commit message: Continued assigning footprints
Parts:
- R36: footprint (none) -> azonenberg_pcb:EIA_0402_RES_NOSILK
Changed lines of the file:
@@
 Sheet 6 12
 Title "FREESAMPLE Oscilloscope"
-Date "2019-03-15"
+Date "2019-03-16"
 Rev "0.1"
 Comp "Andrew D. Zonenberg / Antikernel Labs"
@@
 F 0 "R36" V 1300 3450 50  0000 L CNN
 F 1 "33K" V 1200 3450 50  0000 L CNN
-F 2 "" V 1130 3500 50  0001 C CNN
+F 2 "azonenberg_pcb:EIA_0402_RES_NOSILK" V 1130 3500 50  0001 C CNN
 F 3 "" H 1200 3500 50  0001 C CNN
 	1    1200 3500

Commit message: Continued schematic review. Significantly simplified one-shot to reduce jitter, board area, and power consumption
Parts:
- removed C196, C202, C209: 4.7 uF, azonenberg_pcb:EIA_0603_CAP_NOSILK, symbol device:C
- removed C203, C204, C207, C208: 0.47 uF, azonenberg_pcb:EIA_0402_CAP_NOSILK, symbol device:C
- removed C210, C212: 0.1 uF, azonenberg_pcb:EIA_0402_CAP_NOSILK, symbol device:C
- removed C211, C213: 0.01 uF, azonenberg_pcb:EIA_0402_CAP_NOSILK, symbol device:C
- removed C281, C282, C289, C290, C299, C300, C301, C302, C303, C304, C305, C306: 530Z104KT10T, azonenberg_pcb:EIA_0201_CAP_NOSILK, symbol device:C
- removed JP7: JUMPER_0402, azonenberg_pcb:EIA_0402_JUMPER, symbol special-azonenberg:JUMPER_0402_SPDT
- removed R23: 1K, azonenberg_pcb:EIA_0402_RES_NOSILK, symbol device:R
- removed U23: NB7V52MMNG, azonenberg_pcb:QFN_16_0.5MM_3x3MM, symbol special-azonenberg:NB7V52MMNG
- removed U24: PI6C59S6005, azonenberg_pcb:QFN_24_0.5MM_4x4MM, symbol special-azonenberg:PI6C59S6005
- removed U25: SY58051AU, azonenberg_pcb:QFN_16_0.5MM_3x3MM, symbol special-azonenberg:SY58051AU
Connections:
- net SHREG2B_N is gone; now on net ADC_LE_N: U22.11 (Q4_N)
- net SHREG2B_P is gone; now on net ADC_LE_P: U22.10 (Q4_P)
- net TRG_N: now also U22.24 (Q0_N)
- net TRG_P: now also U22.23 (Q0_P)
- net TRIG_N: now also U22.2 (Q1_N)
- net TRIG_P: now also U22.1 (Q1_P)
- net CLK3_AC_N: no longer names the net of U7.8 (Q3_N)
- net CLK3_AC_P: no longer names the net of U7.7 (Q3_P)
- net RST3_AC_N: no longer names the net of U18.8 (Q3_N)
- net RST3_AC_P: no longer names the net of U18.7 (Q3_P)
- net SHREG2A_N: no longer names the net of U22.8 (Q3_N)
- net SHREG2A_P: no longer names the net of U22.7 (Q3_P)
- no-connect marks 23 -> 17
Other:
- note added: "Comparator:\nLE low: track\nLE high: hold\n\nSo we track during reset\nand latch after a couple of clocks"
- note added: "Register and buffer sampling clock"
- note removed: "Comparator:\nLE low: track\nLE high: hold\n\nSHRE2 & !SHREG3 is the desired track period\nSo we need to invert Q"
- note removed: "Logic function: LE = SHREG2 & !SHREG3"
- note removed: "Shift register for digital one-shot"
- note removed: "Single-cycle pulse output for digital one-shot"
- note removed: "polarity flip = invert"
- moved on the sheet: C311, J17, J18, U40

Commit message: Continued design review. Changed termination on DFFs to 1V8. Added some pull resistors to keep DFFs in reset during boot.
Parts:
- added C196, C202, C203, C204, C207, C208, C209, C210, C211: 0.47 uF, azonenberg_pcb:EIA_0402_CAP_NOSILK, symbol device:C
- added R130: 10K, azonenberg_pcb:EIA_0402_RES_NOSILK, symbol device:R
- added R131, R132, R133, R134, R135, R136: 909, azonenberg_pcb:EIA_0402_RES_NOSILK, symbol device:R
Connections:
- net GND: now also C196.2, C202.2, C203.2, C204.2, C207.2, C208.2, C209.2, C210.2, C211.2, R130.1, R131.1, R133.1, R135.1; no longer U19.13 (VTR), U19.16 (VTR_N), U19.5 (VTCLK), U19.8 (VTCLK_N), U20.1 (VT_D), U20.13 (VTR), U20.16 (VTR_N), U20.4 (VT_D_N), U20.5 (VTCLK), U20.8 (VTCLK_N), U21.1 (VT_D), U21.13 (VTR), U21.16 (VTR_N), U21.4 (VT_D_N), U21.5 (VTCLK), U21.8 (VTCLK_N)
- net RANGE_SEL: now also R130.2
- net RST0_N: now also R131.2
- net RST0_P: now also R132.2
- net RST1_N: now also R133.2
- net RST1_P: now also R134.2
- net RST2_N: now also R135.2
- net RST2_P: now also R136.2
- new net 1V8: C196.1, C202.1, C203.1, C204.1, C207.1, C208.1, C209.1, C210.1, C211.1, R132.1, R134.1, R136.1, U19.13 (VTR), U19.16 (VTR_N), U19.5 (VTCLK), U19.8 (VTCLK_N), U20.1 (VT_D), U20.13 (VTR), U20.16 (VTR_N), U20.4 (VT_D_N), U20.5 (VTCLK), U20.8 (VTCLK_N), U21.1 (VT_D), U21.13 (VTR), U21.16 (VTR_N), U21.4 (VT_D_N), U21.5 (VTCLK), U21.8 (VTCLK_N)
Other:
- note added: "Weakly pull reset inputs of FFs to "reset"\nto prevent self oscillation before FPGA loads\nWe have 50 ohms to 1V8, need to hit 100 mV differential"
- moved on the sheet: JP6

Commit message: Added fiducials
Changed lines of the file:
@@
 	0    1    1    0
 $EndComp
-Text Label 2750 4950 2    50   ~ 0
+Text Label 2750 4950 2    50   ~ 6
 RANGE_SEL
-Text Label 3050 4950 0    50   ~ 0
+Text Label 3050 4950 0    50   ~ 6
 GND
 $Comp
@@
 	0    1    1    0
 $EndComp
-Text Notes 13400 1650 0    50   ~ 0
+Text Notes 13400 1650 0    50   ~ 6
 Weakly pull reset inputs of FFs to "reset"\nto prevent self oscillation before FPGA loads\nWe have 50 ohms to 1V8, need to hit 100 mV differential
-Text Label 13350 1900 2    50   ~ 0
+Text Label 13350 1900 2    50   ~ 6
 RST0_N
-Text Label 13650 1900 0    50   ~ 0
-GND
-Text Label 7100 2250 2    50   ~ 0
-1V8
-Text Label 4050 2550 2    50   ~ 0
-1V8
-Text HLabel 1900 2550 0    50   Input ~ 0
+Text Label 13650 1900 0    50   ~ 6
+GND
+Text Label 7100 2250 2    50   ~ 6
+1V8
+Text Label 4050 2550 2    50   ~ 6
+1V8
+Text HLabel 1900 2550 0    50   Input ~ 6
 1V8
 $Comp
@@
 	1    0    0    -1
 $EndComp
-Text Label 750  650  2    50   ~ 0
+Text Label 750  650  2    50   ~ 6
 1V8
 Wire Wire Line
@@
 	1    0    0    -1
 $EndComp
-Text Label 750  950  2    50   ~ 0
+Text Label 750  950  2    50   ~ 6
 GND
 $Comp
@@
 	0    1    1    0
 $EndComp
-Text Label 13350 2100 2    50   ~ 0
+Text Label 13350 2100 2    50   ~ 6
 RST0_P
-Text Label 13650 2100 0    50   ~ 0
+Text Label 13650 2100 0    50   ~ 6
 1V8
 $Comp
@@
 	0    1    1    0
 $EndComp
-Text Label 13350 2300 2    50   ~ 0
+Text Label 13350 2300 2    50   ~ 6
 RST1_N
-Text Label 13650 2300 0    50   ~ 0
+Text Label 13650 2300 0    50   ~ 6
 GND
 $Comp
@@
 	0    1    1    0
 $EndComp
-Text Label 13350 2500 2    50   ~ 0
+Text Label 13350 2500 2    50   ~ 6
 RST1_P
-Text Label 13650 2500 0    50   ~ 0
+Text Label 13650 2500 0    50   ~ 6
 1V8
 $Comp
@@
 	0    1    1    0
 $EndComp
-Text Label 14200 1900 2    50   ~ 0
+Text Label 14200 1900 2    50   ~ 6
 RST2_N
-Text Label 14500 1900 0    50   ~ 0
+Text Label 14500 1900 0    50   ~ 6
 GND
 $Comp
@@
 	0    1    1    0
 $EndComp
-Text Label 14200 2100 2    50   ~ 0
+Text Label 14200 2100 2    50   ~ 6
 RST2_P
-Text Label 14500 2100 0    50   ~ 0
+Text Label 14500 2100 0    50   ~ 6
 1V8
 $EndSCHEMATC
