File: boards/freesample/oneshot.sch (KiCad schematic (older format))
At the start: 79 parts, among them J17 SMA, J18 SMA, U18 PI6C59S6005, U19 NB7V52MMNG, U20 NB7V52MMNG, U21 NB7V52MMNG, U22 PI6C59S6005, U40 DS25BR150, U7 PI6C59S6005

Commit message: Initial layout work on one-shot. Nowhere near done.
Parts:
- added C212: 0.47 uF, azonenberg_pcb:EIA_0402_CAP_NOSILK, symbol device:C
Connections:
- net 1V8: now also C212.1
- net GND: now also C212.2
Other:
- moved on the sheet: C297, C298, J17, J18, U22
