File: boards/freesample/phase-control.sch (KiCad schematic (older format))
At the start: 43 parts, among them U16 HMC856, U17 NB6L295

Commit message: Began design review. Added review status checklist with current progress. Added some test points, plus an attenuator on the DAC output to prevent bad firmware from damaging the comparators
Parts:
- added R104, R105: 10K, symbol device:R
Connections:
- net COARSE_EN: now also R104.1
- net COARSE_SLOAD: now also R105.1
- net GND: now also R104.2, R105.2
Changed lines of the file:
@@
 Wire Wire Line
 	5950 5950 5950 5750
+$Comp
+L device:R R104
+U 1 1 5D53DE06
+P 5800 6200
+F 0 "R104" V 5700 6200 50  0000 C CNN
+F 1 "10K" V 5800 6200 50  0000 C CNN
+F 2 "" V 5730 6200 50  0001 C CNN
+F 3 "" H 5800 6200 50  0001 C CNN
+	1    5800 6200
+	0    1    1    0
+$EndComp
+Text Label 5650 6200 2    50   ~ 0
+GND
+Text Label 5950 6200 0    50   ~ 0
+COARSE_EN
+$Comp
+L device:R R105
+U 1 1 5D53E277
+P 5800 6400
+F 0 "R105" V 5700 6400 50  0000 C CNN
+F 1 "10K" V 5800 6400 50  0000 C CNN
+F 2 "" V 5730 6400 50  0001 C CNN
+F 3 "" H 5800 6400 50  0001 C CNN
+	1    5800 6400
+	0    1    1    0
+$EndComp
+Wire Wire Line
+	5650 6200 5650 6400
+Text Label 5950 6400 0    50   ~ 0
+COARSE_SLOAD
 $EndSCHEMATC
