File: boards/freesample/freesample.kicad_pcb (KiCad board)
At the start: 8 copper layers, 0 parts

Commit message: Added more test points. Started picking packages for passives. Continued schematic review.
Other:
- net class Default: clearance 0.2 -> 0.1; trace_width 0.25 -> 0.1; via_dia 0.8 -> 0.55; via_drill 0.4 -> 0.3
- rule trace_clearance: 0.2 -> 0.1
- rule trace_min: 0.2 -> 0.1
- rule via_min_drill: 0.3 -> 0.15
- rule via_min_size: 0.4 -> 0.35
Changed lines of the file:
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@@
-(kicad_pcb (version 20171130) (host pcbnew "(6.0.0-rc1-dev-1427-g10887868d)")
+(kicad_pcb (version 20171130) (host pcbnew "(5.1.0)")
   (general
     (thickness 1.6)
@@
   )
   (setup
-    (last_trace_width 0.25)
-    (trace_clearance 0.2)
+    (last_trace_width 0.1)
+    (user_trace_width 0.1)
+    (user_trace_width 0.115)
+    (user_trace_width 0.125)
+    (user_trace_width 0.185)
+    (user_trace_width 0.225)
+    (user_trace_width 0.25)
+    (user_trace_width 0.5)
+    (trace_clearance 0.1)
     (zone_clearance 0.508)
     (zone_45_only no)
-    (trace_min 0.2)
-    (via_size 0.8)
-    (via_drill 0.4)
-    (via_min_size 0.4)
-    (via_min_drill 0.3)
+    (trace_min 0.1)
+    (via_size 0.55)
+    (via_drill 0.3)
+    (via_min_size 0.35)
+    (via_min_drill 0.15)
+    (user_via 0.35 0.15)
+    (user_via 0.55 0.3)
     (uvia_size 0.3)
     (uvia_drill 0.1)
@@
   (net 0 "")
   (net_class Default "This is the default net class."
-    (clearance 0.2)
-    (trace_width 0.25)
-    (via_dia 0.8)
-    (via_drill 0.4)
+    (clearance 0.1)
+    (trace_width 0.1)
+    (via_dia 0.55)
+    (via_drill 0.3)
     (uvia_dia 0.3)
     (uvia_drill 0.1)

Commit message: Initial layout of external refclks block
Parts:
- added C1: 100 pF, azonenberg_pcb:EIA_0201_CAP_NOSILK, F.Cu at (27.6, 142.0)
- added C10: 100 pF, azonenberg_pcb:EIA_0201_CAP_NOSILK, F.Cu at (25.6, 126.2)
- added C100: 0.47 uF, azonenberg_pcb:EIA_0402_CAP_NOSILK, F.Cu at (280.8, 196.6)
- added C101: 0.47 uF, azonenberg_pcb:EIA_0402_CAP_NOSILK, F.Cu at (280.7, 195.1)
- added C102: 0.47 uF, azonenberg_pcb:EIA_0402_CAP_NOSILK, F.Cu at (277.5, 198.6)
- added C103: 4.7 uF, azonenberg_pcb:EIA_0603_CAP_NOSILK, F.Cu at (331.7, 188.1)
- added C104: 4.7 uF, azonenberg_pcb:EIA_0603_CAP_NOSILK, F.Cu at (326.0, 193.2)
- added C105: 4.7 uF, azonenberg_pcb:EIA_0603_CAP_NOSILK, F.Cu at (336.4, 183.4)
- added C106: 4.7 uF, azonenberg_pcb:EIA_0603_CAP_NOSILK, F.Cu at (333.4, 185.5)
- added C107: 4.7 uF, azonenberg_pcb:EIA_0603_CAP_NOSILK, F.Cu at (328.4, 188.1)
- added C108: 4.7 uF, azonenberg_pcb:EIA_0603_CAP_NOSILK, F.Cu at (326.0, 191.4)
- added C109: 0.47 uF, azonenberg_pcb:EIA_0402_CAP_NOSILK, F.Cu at (330.5, 189.7)
- added C11: 100 pF, azonenberg_pcb:EIA_0201_CAP_NOSILK, F.Cu at (30.4, 126.2)
- added C110: 0.47 uF, azonenberg_pcb:EIA_0402_CAP_NOSILK, F.Cu at (328.9, 192.7)
- added C111: 0.47 uF, azonenberg_pcb:EIA_0402_CAP_NOSILK, F.Cu at (331.4, 194.2)
- added C112: 0.47 uF, azonenberg_pcb:EIA_0402_CAP_NOSILK, F.Cu at (328.9, 191.2)
- added C113: 0.47 uF, azonenberg_pcb:EIA_0402_CAP_NOSILK, F.Cu at (331.4, 191.2)
- added C114: 1 uF, azonenberg_pcb:EIA_0402_CAP_NOSILK, F.Cu at (338.8, 185.1)
- added C115: 0.47 uF, azonenberg_pcb:EIA_0402_CAP_NOSILK, F.Cu at (328.9, 194.2)
- added C116: 47 uF, azonenberg_pcb:EIA_1210_CAP_NOSILK, F.Cu at (337.2, 180.6)
- added C117: 0.47 uF, azonenberg_pcb:EIA_0402_CAP_NOSILK, F.Cu at (328.1, 195.7)
- added C118: 0.47 uF, azonenberg_pcb:EIA_0402_CAP_NOSILK, F.Cu at (331.4, 192.7)
- added C119: 27 pF, azonenberg_pcb:EIA_0402_CAP_NOSILK, F.Cu at (337.1, 186.6)
- added C12: 330 pF, azonenberg_pcb:EIA_0201_CAP_NOSILK, F.Cu at (30.0, 122.8)
- added C120: 0.47 uF, azonenberg_pcb:EIA_0402_CAP_NOSILK, F.Cu at (335.5, 188.6)
- added C121: 2700 pF, azonenberg_pcb:EIA_0402_CAP_NOSILK, F.Cu at (333.9, 191.2)
- added C122: 0.47 uF, azonenberg_pcb:EIA_0402_CAP_NOSILK, F.Cu at (339.6, 186.6)
- added C123: 0.47 uF, azonenberg_pcb:EIA_0402_CAP_NOSILK, F.Cu at (333.0, 189.7)
- added C124: 0.47 uF, azonenberg_pcb:EIA_0402_CAP_NOSILK, F.Cu at (328.0, 189.7)
- added C125: 0.47 uF, azonenberg_pcb:EIA_0402_CAP_NOSILK, F.Cu at (336.3, 185.1)
- added C126: 0.47 uF, azonenberg_pcb:EIA_0402_CAP_NOSILK, F.Cu at (325.6, 194.9)
- added C127: 10 uF, azonenberg_pcb:EIA_1206_CAP_NOSILK, F.Cu at (329.2, 185.9)
- added C128: 0.1 uF, azonenberg_pcb:EIA_0402_CAP_NOSILK, F.Cu at (339.3, 183.3)
- added C129: 0.1 uF, azonenberg_pcb:EIA_0402_CAP_NOSILK, F.Cu at (255.0, 211.0)
- added C13: 330 pF, azonenberg_pcb:EIA_0201_CAP_NOSILK, F.Cu at (25.4, 145.9)
- added C130: 0.1 uF, azonenberg_pcb:EIA_0402_CAP_NOSILK, F.Cu at (247.5, 211.0)
- added C131: 0.1 uF, azonenberg_pcb:EIA_0402_CAP_NOSILK, F.Cu at (238.7, 184.5)
- added C132: 0.1 uF, azonenberg_pcb:EIA_0402_CAP_NOSILK, F.Cu at (250.0, 211.0)
- added C133: 100 pF, azonenberg_pcb:EIA_0201_CAP_NOSILK, F.Cu at (337.4, 229.9)
- added C134: 100 pF, azonenberg_pcb:EIA_0201_CAP_NOSILK, F.Cu at (335.8, 234.7)
- added C135: 100 pF, azonenberg_pcb:EIA_0201_CAP_NOSILK, F.Cu at (338.3, 231.4)
- added C136: 100 pF, azonenberg_pcb:EIA_0201_CAP_NOSILK, F.Cu at (336.6, 236.2)
- added C137: 100 pF, azonenberg_pcb:EIA_0201_CAP_NOSILK, F.Cu at (337.4, 234.7)
- added C138: 330 pF, azonenberg_pcb:EIA_0201_CAP_NOSILK, F.Cu at (334.9, 236.2)
- added C139: 330 pF, azonenberg_pcb:EIA_0201_CAP_NOSILK, F.Cu at (337.4, 233.2)
- added C14: 330 pF, azonenberg_pcb:EIA_0201_CAP_NOSILK, F.Cu at (31.5, 143.8)
- added C140: 330 pF, azonenberg_pcb:EIA_0201_CAP_NOSILK, F.Cu at (336.6, 231.7)
- added C141: 4.7 uF, azonenberg_pcb:EIA_0603_CAP_NOSILK, F.Cu at (330.8, 234.5)
- added C142: 4.7 uF, azonenberg_pcb:EIA_0603_CAP_NOSILK, F.Cu at (326.0, 234.9)
- added C143: 4.7 uF, azonenberg_pcb:EIA_0603_CAP_NOSILK, F.Cu at (334.9, 230.1)
- added C144: 100 pF, azonenberg_pcb:EIA_0201_CAP_NOSILK, F.Cu at (333.3, 235.8)
- added C145: 4.7 uF, azonenberg_pcb:EIA_0603_CAP_NOSILK, F.Cu at (327.2, 202.7)
- added C146: 530Z104KT10T, azonenberg_pcb:EIA_0201_CAP_NOSILK, F.Cu at (330.5, 205.6)
- added C147: 530Z104KT10T, azonenberg_pcb:EIA_0201_CAP_NOSILK, F.Cu at (328.0, 208.8)
- added C148: 530Z104KT10T, azonenberg_pcb:EIA_0201_CAP_NOSILK, F.Cu at (324.7, 211.8)
- added C149: 530Z104KT10T, azonenberg_pcb:EIA_0201_CAP_NOSILK, F.Cu at (330.0, 201.1)
- added C15: 4.7 uF, azonenberg_pcb:EIA_0603_CAP_NOSILK, F.Cu at (32.3, 142.8)
- added C150: 0.47 uF, azonenberg_pcb:EIA_0402_CAP_NOSILK, F.Cu at (330.1, 202.6)
- added C151: 0.47 uF, azonenberg_pcb:EIA_0402_CAP_NOSILK, F.Cu at (326.0, 208.8)
- added C152: 0.47 uF, azonenberg_pcb:EIA_0402_CAP_NOSILK, F.Cu at (326.0, 207.3)
- added C153: 0.47 uF, azonenberg_pcb:EIA_0402_CAP_NOSILK, F.Cu at (328.5, 205.8)
- added C154: 0.01 uF, azonenberg_pcb:EIA_0402_CAP_NOSILK, F.Cu at (328.5, 204.3)
- added C155: 530Z104KT10T, azonenberg_pcb:EIA_0201_CAP_NOSILK, F.Cu at (325.5, 210.3)
- added C156: 530Z104KT10T, azonenberg_pcb:EIA_0201_CAP_NOSILK, F.Cu at (330.5, 204.1)
- added C157: 0.01 uF, azonenberg_pcb:EIA_0402_CAP_NOSILK, F.Cu at (323.5, 210.3)
- added C158: 4.7 uF, azonenberg_pcb:EIA_0603_CAP_NOSILK, F.Cu at (323.9, 202.7)
- added C159: 0.47 uF, azonenberg_pcb:EIA_0402_CAP_NOSILK, F.Cu at (323.5, 204.3)
- added C16: 530Z104KT10T, azonenberg_pcb:EIA_0201_CAP_NOSILK, F.Cu at (25.0, 144.2)
- added C160: 0.47 uF, azonenberg_pcb:EIA_0402_CAP_NOSILK, F.Cu at (323.5, 208.8)
- added C161: 0.47 uF, azonenberg_pcb:EIA_0402_CAP_NOSILK, F.Cu at (326.0, 205.8)
- added C162: 0.47 uF, azonenberg_pcb:EIA_0402_CAP_NOSILK, F.Cu at (326.0, 204.3)
- added C163: 4.7 uF, azonenberg_pcb:EIA_0603_CAP_NOSILK, F.Cu at (307.7, 233.1)
- added C164: 4.7 uF, azonenberg_pcb:EIA_0603_CAP_NOSILK, F.Cu at (303.9, 234.1)
- added C165: 100 pF, azonenberg_pcb:EIA_0201_CAP_NOSILK, F.Cu at (318.0, 229.8)
- added C166: 0.47 uF, azonenberg_pcb:EIA_0402_CAP_NOSILK, F.Cu at (302.7, 237.2)
- added C167: 0.47 uF, azonenberg_pcb:EIA_0402_CAP_NOSILK, F.Cu at (313.5, 228.2)
- added C168: 100 pF, azonenberg_pcb:EIA_0201_CAP_NOSILK, F.Cu at (315.2, 232.8)
- added C169: 0.47 uF, azonenberg_pcb:EIA_0402_CAP_NOSILK, F.Cu at (300.2, 235.7)
- added C17: 530Z104KT10T, azonenberg_pcb:EIA_0201_CAP_NOSILK, F.Cu at (25.0, 144.8)
- added C170: 0.47 uF, azonenberg_pcb:EIA_0402_CAP_NOSILK, F.Cu at (313.5, 229.8)
- added C171: 0.47 uF, azonenberg_pcb:EIA_0402_CAP_NOSILK, F.Cu at (305.2, 236.2)
- added C172: 0.47 uF, azonenberg_pcb:EIA_0402_CAP_NOSILK, F.Cu at (305.2, 237.7)
- added C173: 100 pF, azonenberg_pcb:EIA_0201_CAP_NOSILK, F.Cu at (318.0, 228.2)
- added C174: 100 pF, azonenberg_pcb:EIA_0201_CAP_NOSILK, F.Cu at (317.1, 234.2)
- added C175: 4.7 uF, azonenberg_pcb:EIA_0603_CAP_NOSILK, F.Cu at (300.6, 234.1)
- added C176: 4.7 uF, azonenberg_pcb:EIA_0603_CAP_NOSILK, F.Cu at (281.3, 214.0)
- added C177: 530Z104KT10T, azonenberg_pcb:EIA_0201_CAP_NOSILK, F.Cu at (287.6, 220.2)
- added C178: 530Z104KT10T, azonenberg_pcb:EIA_0201_CAP_NOSILK, F.Cu at (292.4, 215.4)
- added C179: 530Z104KT10T, azonenberg_pcb:EIA_0201_CAP_NOSILK, F.Cu at (297.1, 210.6)
- added C18: 330 pF, azonenberg_pcb:EIA_0201_CAP_NOSILK, F.Cu at (28.5, 127.7)
- added C180: 530Z104KT10T, azonenberg_pcb:EIA_0201_CAP_NOSILK, F.Cu at (285.1, 221.7)
- added C181: 0.01 uF, azonenberg_pcb:EIA_0402_CAP_NOSILK, F.Cu at (295.5, 206.1)
- added C182: 0.47 uF, azonenberg_pcb:EIA_0402_CAP_NOSILK, F.Cu at (281.4, 220.1)
- added C183: 0.47 uF, azonenberg_pcb:EIA_0402_CAP_NOSILK, F.Cu at (286.2, 215.7)
- added C184: 0.47 uF, azonenberg_pcb:EIA_0402_CAP_NOSILK, F.Cu at (290.0, 212.4)
- added C185: 0.47 uF, azonenberg_pcb:EIA_0402_CAP_NOSILK, F.Cu at (288.5, 209.4)
- added C186: 4.7 uF, azonenberg_pcb:EIA_0603_CAP_NOSILK, F.Cu at (285.4, 211.1)
- added C187: 0.01 uF, azonenberg_pcb:EIA_0402_CAP_NOSILK, F.Cu at (281.2, 217.1)
- added C188: 0.47 uF, azonenberg_pcb:EIA_0402_CAP_NOSILK, F.Cu at (293.0, 207.9)
- added C189: 0.47 uF, azonenberg_pcb:EIA_0402_CAP_NOSILK, F.Cu at (282.7, 218.6)
- added C19: 330 pF, azonenberg_pcb:EIA_0201_CAP_NOSILK, F.Cu at (31.4, 124.6)
- added C190: 0.47 uF, azonenberg_pcb:EIA_0402_CAP_NOSILK, F.Cu at (288.3, 210.9)
- added C191: 0.47 uF, azonenberg_pcb:EIA_0402_CAP_NOSILK, F.Cu at (283.7, 217.1)
- added C192: 0.47 uF, azonenberg_pcb:EIA_0402_CAP_NOSILK, F.Cu at (296.3, 204.6)
- added C193: 0.47 uF, azonenberg_pcb:EIA_0402_CAP_NOSILK, F.Cu at (287.5, 212.7)
- added C194: 0.47 uF, azonenberg_pcb:EIA_0402_CAP_NOSILK, F.Cu at (291.0, 209.4)
- added C195: 0.47 uF, azonenberg_pcb:EIA_0402_CAP_NOSILK, F.Cu at (290.5, 207.9)
- added C196: 0.47 uF, azonenberg_pcb:EIA_0402_CAP_NOSILK, F.Cu at (280.2, 218.6)
- added C197: 4.7 uF, azonenberg_pcb:EIA_0603_CAP_NOSILK, F.Cu at (290.9, 204.8)
- added C198: 0.47 uF, azonenberg_pcb:EIA_0402_CAP_NOSILK, F.Cu at (283.7, 215.6)
- added C199: 0.47 uF, azonenberg_pcb:EIA_0402_CAP_NOSILK, F.Cu at (293.0, 206.4)
- added C2: 100 pF, azonenberg_pcb:EIA_0201_CAP_NOSILK, F.Cu at (30.5, 145.5)
- added C20: 4.7 uF, azonenberg_pcb:EIA_0603_CAP_NOSILK, F.Cu at (32.2, 123.7)
- added C200: 0.47 uF, azonenberg_pcb:EIA_0402_CAP_NOSILK, F.Cu at (286.2, 214.2)
- added C201: 0.47 uF, azonenberg_pcb:EIA_0402_CAP_NOSILK, F.Cu at (278.9, 221.4)
- added C202: 0.47 uF, azonenberg_pcb:EIA_0402_CAP_NOSILK, F.Cu at (277.7, 219.9)
- added C203: 0.47 uF, azonenberg_pcb:EIA_0402_CAP_NOSILK, F.Cu at (277.7, 218.4)
- added C204: 0.47 uF, azonenberg_pcb:EIA_0402_CAP_NOSILK, F.Cu at (276.4, 221.7)
- added C205: 530Z104KT10T, azonenberg_pcb:EIA_0201_CAP_NOSILK, F.Cu at (323.0, 211.8)
- added C206: 530Z104KT10T, azonenberg_pcb:EIA_0201_CAP_NOSILK, F.Cu at (328.0, 207.3)
- added C207: 0.47 uF, azonenberg_pcb:EIA_0402_CAP_NOSILK, F.Cu at (285.0, 212.7)
- added C208: 0.47 uF, azonenberg_pcb:EIA_0402_CAP_NOSILK, F.Cu at (290.5, 206.4)
- added C209: 0.47 uF, azonenberg_pcb:EIA_0402_CAP_NOSILK, F.Cu at (281.2, 215.6)
- added C21: 4.7 uF, azonenberg_pcb:EIA_0603_CAP_NOSILK, F.Cu at (27.1, 148.2)
- added C210: 0.47 uF, azonenberg_pcb:EIA_0402_CAP_NOSILK, F.Cu at (293.8, 204.6)
- added C211: 0.47 uF, azonenberg_pcb:EIA_0402_CAP_NOSILK, F.Cu at (290.8, 210.9)
- added C214: 1 uF, azonenberg_pcb:EIA_0603_CAP_NOSILK, F.Cu at (282.8, 279.1)
- added C215: 1 uF, azonenberg_pcb:EIA_0603_CAP_NOSILK, F.Cu at (277.1, 281.5)
- added C216: 0.1 uF, azonenberg_pcb:EIA_0402_CAP_NOSILK, F.Cu at (292.0, 275.1)
- added C217: 0.01 uF, azonenberg_pcb:EIA_0402_CAP_NOSILK, F.Cu at (287.5, 280.4)
- added C218: 0.1 uF, azonenberg_pcb:EIA_0402_CAP_NOSILK, F.Cu at (292.0, 276.6)
- added C219: 4.7 uF 12V, azonenberg_pcb:EIA_1206_CAP_NOSILK, F.Cu at (210.5, 267.2)
- added C22: 4.7 uF, azonenberg_pcb:EIA_0603_CAP_NOSILK, F.Cu at (32.3, 145.4)
- added C220: 4.7 uF 5V, azonenberg_pcb:EIA_1206_CAP_NOSILK, F.Cu at (222.5, 167.4)
- added C221: 4.7 uF 5V, azonenberg_pcb:EIA_1206_CAP_NOSILK, F.Cu at (239.0, 238.4)
- added C222: 4.7 uF 5V, azonenberg_pcb:EIA_1206_CAP_NOSILK, F.Cu at (246.0, 232.3)
- added C223: 2.2 uF 5V, azonenberg_pcb:EIA_0603_CAP_NOSILK, F.Cu at (233.6, 249.5)
- added C224: 1 uF 5V, azonenberg_pcb:EIA_0603_CAP_NOSILK, F.Cu at (223.1, 259.2)
- added C225: 4.7 uF, azonenberg_pcb:EIA_0603_CAP_NOSILK, F.Cu at (246.5, 238.2)
- added C226: 1 uF, azonenberg_pcb:EIA_0603_CAP_NOSILK, F.Cu at (251.0, 234.3)
- added C227: 22 nF, azonenberg_pcb:EIA_0402_CAP_NOSILK, F.Cu at (226.0, 260.4)
- added C228: 22 uF, azonenberg_pcb:EIA_0805_CAP_NOSILK, F.Cu at (207.7, 249.0)
- added C229: 1 uF, azonenberg_pcb:EIA_0603_CAP_NOSILK, F.Cu at (241.3, 244.2)
- added C23: 4.7 uF, azonenberg_pcb:EIA_0603_CAP_NOSILK, F.Cu at (27.1, 128.7)
- added C230: 4.7 uF, azonenberg_pcb:EIA_0603_CAP_NOSILK, F.Cu at (223.1, 262.8)
- added C231: 1 uF, azonenberg_pcb:EIA_0402_CAP_NOSILK, F.Cu at (244.2, 243.2)
- added C232: 22 uF, azonenberg_pcb:EIA_0805_CAP_NOSILK, F.Cu at (214.8, 266.1)
- added C233: 22 uF, azonenberg_pcb:EIA_0805_CAP_NOSILK, F.Cu at (250.3, 232.1)
- added C234: 22 uF, azonenberg_pcb:EIA_0805_CAP_NOSILK, F.Cu at (235.0, 247.3)
- added C235: 22 uF 16V, azonenberg_pcb:EIA_1812_CAP_NOSILK, F.Cu at (205.4, 257.8)
- added C236: 22 uF 10V, azonenberg_pcb:EIA_1210_CAP_NOSILK, F.Cu at (239.8, 235.2)
- added C237: 22 uF 16V, azonenberg_pcb:EIA_1812_CAP_NOSILK, F.Cu at (233.9, 229.1)
- added C238: 22 uF 10V, azonenberg_pcb:EIA_1210_CAP_NOSILK, F.Cu at (246.0, 229.0)
- added C239: 10 nF, azonenberg_pcb:EIA_0402_CAP_NOSILK, F.Cu at (250.6, 236.0)
- added C24: 4.7 uF, azonenberg_pcb:EIA_0603_CAP_NOSILK, F.Cu at (32.2, 126.2)
- added C240: 22 uF 16V, azonenberg_pcb:EIA_1812_CAP_NOSILK, F.Cu at (233.9, 233.1)
- added C241: 4.7 uF, azonenberg_pcb:EIA_0603_CAP_NOSILK, F.Cu at (241.3, 240.6)
- added C242: 4.7 uF, azonenberg_pcb:EIA_0603_CAP_NOSILK, F.Cu at (243.2, 238.2)
- added C243: 22 uF 16V, azonenberg_pcb:EIA_1812_CAP_NOSILK, F.Cu at (225.7, 239.4)
- added C244: 10 nF, azonenberg_pcb:EIA_0402_CAP_NOSILK, F.Cu at (238.1, 248.6)
- added C245: 10 nF, azonenberg_pcb:EIA_0402_CAP_NOSILK, F.Cu at (244.2, 241.7)
- added C246: 4.7 uF, azonenberg_pcb:EIA_0603_CAP_NOSILK, F.Cu at (218.3, 265.7)
- added C247: 4.7 uF, azonenberg_pcb:EIA_0603_CAP_NOSILK, F.Cu at (229.7, 252.9)
- added C248: 4.7 uF, azonenberg_pcb:EIA_0603_CAP_NOSILK, F.Cu at (223.1, 261.0)
- added C249: 4.7 uF, azonenberg_pcb:EIA_0603_CAP_NOSILK, F.Cu at (244.6, 240.0)
- added C25: 100 pF, azonenberg_pcb:EIA_0201_CAP_NOSILK, F.Cu at (27.5, 147.0)
- added C250: 22 uF 16V, azonenberg_pcb:EIA_1812_CAP_NOSILK, F.Cu at (213.6, 249.7)
- added C251: 22 uF 10V, azonenberg_pcb:EIA_1210_CAP_NOSILK, F.Cu at (214.8, 262.8)
- added C252: 22 uF 16V, azonenberg_pcb:EIA_1812_CAP_NOSILK, F.Cu at (225.7, 243.4)
- added C253: 4.7 uF 5V, azonenberg_pcb:EIA_1206_CAP_NOSILK, F.Cu at (230.7, 246.9)
- added C254: 4.7 uF 5V, azonenberg_pcb:EIA_1206_CAP_NOSILK, F.Cu at (214.8, 259.5)
- added C255: 22 uF 10V, azonenberg_pcb:EIA_1210_CAP_NOSILK, F.Cu at (225.7, 247.3)
- added C256: 2.2 uF 5V, azonenberg_pcb:EIA_0603_CAP_NOSILK, F.Cu at (247.7, 236.3)
- added C257: 1 uF 5V, azonenberg_pcb:EIA_0603_CAP_NOSILK, F.Cu at (229.7, 254.7)
- added C258: 4.7 uF 5V, azonenberg_pcb:EIA_1206_CAP_NOSILK, F.Cu at (205.5, 267.4)
- added C259: 4.7 uF 5V, azonenberg_pcb:EIA_1206_CAP_NOSILK, F.Cu at (225.7, 250.6)
- added C26: 100 pF, azonenberg_pcb:EIA_0201_CAP_NOSILK, F.Cu at (27.5, 122.8)
- added C260: 2.2 uF 5V, azonenberg_pcb:EIA_0603_CAP_NOSILK, F.Cu at (253.8, 229.8)
- added C261: 1 uF 5V, azonenberg_pcb:EIA_0603_CAP_NOSILK, F.Cu at (241.3, 242.4)
- added C262: 0.01 uF, azonenberg_pcb:EIA_0402_CAP_NOSILK, F.Cu at (339.8, 217.3)
- added C263: 530Z104KT10T, azonenberg_pcb:EIA_0201_CAP_NOSILK, F.Cu at (309.7, 237.7)
- added C264: 530Z104KT10T, azonenberg_pcb:EIA_0201_CAP_NOSILK, F.Cu at (319.7, 228.2)
- added C265: 530Z104KT10T, azonenberg_pcb:EIA_0201_CAP_NOSILK, F.Cu at (315.5, 231.2)
- added C266: 530Z104KT10T, azonenberg_pcb:EIA_0201_CAP_NOSILK, F.Cu at (312.2, 235.9)
- added C267: 530Z104KT10T, azonenberg_pcb:EIA_0201_CAP_NOSILK, F.Cu at (317.2, 231.2)
- added C268: 530Z104KT10T, azonenberg_pcb:EIA_0201_CAP_NOSILK, F.Cu at (311.4, 237.7)
- added C269: 530Z104KT10T, azonenberg_pcb:EIA_0201_CAP_NOSILK, F.Cu at (316.8, 232.8)
- added C27: 0.01 uF, azonenberg_pcb:EIA_0402_CAP_NOSILK, B.Cu at (37.5, 133.8)
- added C270: 530Z104KT10T, azonenberg_pcb:EIA_0201_CAP_NOSILK, F.Cu at (319.7, 229.8)
- added C271: 530Z104KT10T, azonenberg_pcb:EIA_0201_CAP_NOSILK, F.Cu at (315.5, 234.2)
- added C272: 530Z104KT10T, azonenberg_pcb:EIA_0201_CAP_NOSILK, F.Cu at (313.9, 235.9)
- added C273: 530Z104KT10T, azonenberg_pcb:EIA_0201_CAP_NOSILK, F.Cu at (318.8, 231.2)
- added C274: 530Z104KT10T, azonenberg_pcb:EIA_0201_CAP_NOSILK, F.Cu at (313.0, 237.4)
- added C275: 530Z104KT10T, azonenberg_pcb:EIA_0201_CAP_NOSILK, F.Cu at (290.8, 215.4)
- added C276: 530Z104KT10T, azonenberg_pcb:EIA_0201_CAP_NOSILK, F.Cu at (294.1, 215.4)
- added C277: 530Z104KT10T, azonenberg_pcb:EIA_0201_CAP_NOSILK, F.Cu at (291.6, 216.9)
- added C278: 530Z104KT10T, azonenberg_pcb:EIA_0201_CAP_NOSILK, F.Cu at (296.3, 212.4)
- added C279: 530Z104KT10T, azonenberg_pcb:EIA_0201_CAP_NOSILK, F.Cu at (286.8, 221.7)
- added C28: 530Z104KT10T, azonenberg_pcb:EIA_0201_CAP_NOSILK, F.Cu at (35.9, 131.6)
- added C280: 530Z104KT10T, azonenberg_pcb:EIA_0201_CAP_NOSILK, F.Cu at (294.1, 213.9)
- added C283: 530Z104KT10T, azonenberg_pcb:EIA_0201_CAP_NOSILK, F.Cu at (289.3, 218.7)
- added C284: 530Z104KT10T, azonenberg_pcb:EIA_0201_CAP_NOSILK, F.Cu at (289.9, 217.2)
- added C285: 530Z104KT10T, azonenberg_pcb:EIA_0201_CAP_NOSILK, F.Cu at (298.4, 204.6)
- added C286: 530Z104KT10T, azonenberg_pcb:EIA_0201_CAP_NOSILK, F.Cu at (283.5, 221.6)
- added C287: 530Z104KT10T, azonenberg_pcb:EIA_0201_CAP_NOSILK, F.Cu at (297.6, 207.6)
- added C288: 530Z104KT10T, azonenberg_pcb:EIA_0201_CAP_NOSILK, F.Cu at (295.4, 210.9)
- added C29: 530Z104KT10T, azonenberg_pcb:EIA_0201_CAP_NOSILK, F.Cu at (35.5, 131.9)
- added C291: 530Z104KT10T, azonenberg_pcb:EIA_0201_CAP_NOSILK, F.Cu at (318.5, 232.8)
- added C292: 530Z104KT10T, azonenberg_pcb:EIA_0201_CAP_NOSILK, F.Cu at (313.8, 234.4)
- added C293: 530Z104KT10T, azonenberg_pcb:EIA_0201_CAP_NOSILK, F.Cu at (298.1, 209.1)
- added C294: 530Z104KT10T, azonenberg_pcb:EIA_0201_CAP_NOSILK, F.Cu at (294.6, 212.4)
- added C295: 530Z104KT10T, azonenberg_pcb:EIA_0201_CAP_NOSILK, F.Cu at (292.4, 213.9)
- added C296: 530Z104KT10T, azonenberg_pcb:EIA_0201_CAP_NOSILK, F.Cu at (289.3, 220.2)
- added C297: 530Z104KT10T, azonenberg_pcb:EIA_0201_CAP_NOSILK, F.Cu at (287.6, 218.7)
- added C298: 530Z104KT10T, azonenberg_pcb:EIA_0201_CAP_NOSILK, F.Cu at (286.0, 220.2)
- added C3: 100 pF, azonenberg_pcb:EIA_0201_CAP_NOSILK, F.Cu at (28.9, 142.0)
- added C30: 530Z104KT10T, azonenberg_pcb:EIA_0201_CAP_NOSILK, F.Cu at (35.0, 137.2)
- added C307: 530Z104KT10T, azonenberg_pcb:EIA_0201_CAP_NOSILK, F.Cu at (286.0, 218.7)
- added C308: 530Z104KT10T, azonenberg_pcb:EIA_0201_CAP_NOSILK, F.Cu at (288.3, 217.2)
- added C309: 530Z104KT10T, azonenberg_pcb:EIA_0201_CAP_NOSILK, F.Cu at (331.0, 236.1)
- added C31: 530Z104KT10T, azonenberg_pcb:EIA_0201_CAP_NOSILK, F.Cu at (35.3, 137.6)
- added C310: 530Z104KT10T, azonenberg_pcb:EIA_0201_CAP_NOSILK, F.Cu at (335.8, 233.2)
- added C311: 0.47 uF, azonenberg_pcb:EIA_0402_CAP_NOSILK, F.Cu at (296.0, 209.1)
- added C312: 0.47 uF, azonenberg_pcb:EIA_0402_CAP_NOSILK, F.Cu at (333.7, 234.3)
- added C313: 530Z104KT10T, azonenberg_pcb:EIA_0201_CAP_NOSILK, F.Cu at (290.8, 213.9)
- added C314: 530Z104KT10T, azonenberg_pcb:EIA_0201_CAP_NOSILK, F.Cu at (290.9, 218.7)
- added C315: 10 nF, azonenberg_pcb:EIA_0402_CAP_NOSILK, F.Cu at (232.6, 254.5)
- added C316: 10 nF, azonenberg_pcb:EIA_0402_CAP_NOSILK, F.Cu at (228.2, 257.4)
- added C317: 4.7 uF, azonenberg_pcb:EIA_0603_CAP_NOSILK, F.Cu at (219.0, 263.6)
- added C318: 4.7 uF, azonenberg_pcb:EIA_0603_CAP_NOSILK, F.Cu at (238.5, 246.9)
- added C319: 4.7 uF, azonenberg_pcb:EIA_0603_CAP_NOSILK, F.Cu at (233.6, 251.3)
- added C32: 4.7 uF, azonenberg_pcb:EIA_0603_CAP_NOSILK, F.Cu at (38.8, 139.9)
- added C320: 4.7 uF, azonenberg_pcb:EIA_0603_CAP_NOSILK, F.Cu at (253.7, 231.7)
- added C321: 0.1 uF, azonenberg_pcb:EIA_0402_CAP_NOSILK, F.Cu at (245.0, 211.0)
- added C324: 1 uF, azonenberg_pcb:EIA_0603_CAP_NOSILK, F.Cu at (292.4, 271.9)
- added C325: 0.1 uF, azonenberg_pcb:EIA_0402_CAP_NOSILK, F.Cu at (280.0, 281.3)
- added C326: 0.1 uF, azonenberg_pcb:EIA_0402_CAP_NOSILK, F.Cu at (285.7, 278.9)
- added C33: 0.47 uF, azonenberg_pcb:EIA_0402_CAP_NOSILK, F.Cu at (42.6, 136.0)
- added C34: 0.47 uF, azonenberg_pcb:EIA_0402_CAP_NOSILK, F.Cu at (41.4, 137.8)
- added C35: 0.47 uF, azonenberg_pcb:EIA_0402_CAP_NOSILK, F.Cu at (41.8, 132.6)
- added C36: 0.47 uF, azonenberg_pcb:EIA_0402_CAP_NOSILK, F.Cu at (37.1, 137.9)
- added C37: 100 pF, azonenberg_pcb:EIA_0201_CAP_NOSILK, F.Cu at (338.8, 222.1)
- added C38: 100 pF, azonenberg_pcb:EIA_0201_CAP_NOSILK, F.Cu at (340.3, 220.3)
- added C39: 100 pF, azonenberg_pcb:EIA_0201_CAP_NOSILK, F.Cu at (337.1, 223.6)
- added C4: 100 pF, azonenberg_pcb:EIA_0201_CAP_NOSILK, F.Cu at (27.5, 127.7)
- added C40: 100 pF, azonenberg_pcb:EIA_0201_CAP_NOSILK, F.Cu at (340.3, 218.8)
- added C41: 100 pF, azonenberg_pcb:EIA_0201_CAP_NOSILK, F.Cu at (338.6, 219.1)
- added C42: 330 pF, azonenberg_pcb:EIA_0201_CAP_NOSILK, F.Cu at (336.1, 220.6)
- added C43: 330 pF, azonenberg_pcb:EIA_0201_CAP_NOSILK, F.Cu at (332.0, 225.4)
- added C44: 330 pF, azonenberg_pcb:EIA_0201_CAP_NOSILK, F.Cu at (337.1, 222.1)
- added C45: 4.7 uF, azonenberg_pcb:EIA_0603_CAP_NOSILK, F.Cu at (332.1, 222.2)
- added C46: 4.7 uF, azonenberg_pcb:EIA_0603_CAP_NOSILK, F.Cu at (336.9, 217.4)
- added C47: 4.7 uF, azonenberg_pcb:EIA_0603_CAP_NOSILK, F.Cu at (329.5, 224.1)
- added C48: 100 pF, azonenberg_pcb:EIA_0201_CAP_NOSILK, F.Cu at (337.8, 220.6)
- added C49: 530Z104KT10T, azonenberg_pcb:EIA_0201_CAP_NOSILK, F.Cu at (333.6, 225.4)
- added C5: 100 pF, azonenberg_pcb:EIA_0201_CAP_NOSILK, F.Cu at (30.4, 124.3)
- added C50: 530Z104KT10T, azonenberg_pcb:EIA_0201_CAP_NOSILK, F.Cu at (335.3, 225.1)
- added C51: 4.7 uF, azonenberg_pcb:EIA_0603_CAP_NOSILK, F.Cu at (326.0, 225.1)
- added C52: 0.47 uF, azonenberg_pcb:EIA_0402_CAP_NOSILK, F.Cu at (335.0, 223.6)
- added C53: 0.47 uF, azonenberg_pcb:EIA_0402_CAP_NOSILK, F.Cu at (336.5, 219.1)
- added C54: 0.47 uF, azonenberg_pcb:EIA_0402_CAP_NOSILK, F.Cu at (332.4, 223.9)
- added C55: 0.47 uF, azonenberg_pcb:EIA_0402_CAP_NOSILK, F.Cu at (335.0, 222.1)
- added C56: 530Z104KT10T, azonenberg_pcb:EIA_0201_CAP_NOSILK, F.Cu at (282.9, 196.0)
- added C57: 530Z104KT10T, azonenberg_pcb:EIA_0201_CAP_NOSILK, F.Cu at (285.4, 194.5)
- added C58: 0.47 uF, azonenberg_pcb:EIA_0402_CAP_NOSILK, F.Cu at (278.3, 196.6)
- added C59: 4.7 uF, azonenberg_pcb:EIA_0603_CAP_NOSILK, F.Cu at (270.4, 197.3)
- added C6: 100 pF, azonenberg_pcb:EIA_0201_CAP_NOSILK, F.Cu at (29.0, 122.8)
- added C60: 0.47 uF, azonenberg_pcb:EIA_0402_CAP_NOSILK, F.Cu at (270.0, 195.0)
- added C61: 530Z104KT10T, azonenberg_pcb:EIA_0201_CAP_NOSILK, F.Cu at (294.6, 194.5)
- added C62: 530Z104KT10T, azonenberg_pcb:EIA_0201_CAP_NOSILK, F.Cu at (299.8, 190.2)
- added C63: 530Z104KT10T, azonenberg_pcb:EIA_0201_CAP_NOSILK, F.Cu at (294.6, 196.0)
- added C64: 530Z104KT10T, azonenberg_pcb:EIA_0201_CAP_NOSILK, F.Cu at (292.1, 199.0)
- added C65: 530Z104KT10T, azonenberg_pcb:EIA_0201_CAP_NOSILK, F.Cu at (296.3, 194.5)
- added C66: 530Z104KT10T, azonenberg_pcb:EIA_0201_CAP_NOSILK, F.Cu at (302.3, 188.7)
- added C67: 4.7 uF, azonenberg_pcb:EIA_0603_CAP_NOSILK, F.Cu at (273.6, 191.2)
- added C68: 4.7 uF, azonenberg_pcb:EIA_0603_CAP_NOSILK, F.Cu at (267.1, 195.2)
- added C69: 4.7 uF, azonenberg_pcb:EIA_0603_CAP_NOSILK, F.Cu at (278.6, 188.6)
- added C7: 100 pF, azonenberg_pcb:EIA_0201_CAP_NOSILK, F.Cu at (28.5, 147.0)
- added C70: 4.7 uF, azonenberg_pcb:EIA_0603_CAP_NOSILK, F.Cu at (281.9, 188.6)
- added C71: 4.7 uF, azonenberg_pcb:EIA_0603_CAP_NOSILK, F.Cu at (300.6, 179.5)
- added C72: 4.7 uF, azonenberg_pcb:EIA_0603_CAP_NOSILK, F.Cu at (267.1, 197.0)
- added C73: 4.7 uF, azonenberg_pcb:EIA_0603_CAP_NOSILK, F.Cu at (278.6, 186.8)
- added C74: 4.7 uF, azonenberg_pcb:EIA_0603_CAP_NOSILK, F.Cu at (273.6, 189.4)
- added C75: 0.47 uF, azonenberg_pcb:EIA_0402_CAP_NOSILK, F.Cu at (290.0, 197.5)
- added C76: 4.7 uF, azonenberg_pcb:EIA_0603_CAP_NOSILK, F.Cu at (276.9, 190.4)
- added C77: 4.7 uF, azonenberg_pcb:EIA_0603_CAP_NOSILK, F.Cu at (281.9, 186.8)
- added C78: 4.7 uF, azonenberg_pcb:EIA_0603_CAP_NOSILK, F.Cu at (267.1, 198.8)
- added C79: 0.47 uF, azonenberg_pcb:EIA_0402_CAP_NOSILK, F.Cu at (300.2, 187.2)
- added C8: 100 pF, azonenberg_pcb:EIA_0201_CAP_NOSILK, F.Cu at (30.5, 143.5)
- added C80: 0.47 uF, azonenberg_pcb:EIA_0402_CAP_NOSILK, F.Cu at (287.5, 199.0)
- added C81: 0.47 uF, azonenberg_pcb:EIA_0402_CAP_NOSILK, F.Cu at (292.5, 194.5)
- added C82: 0.47 uF, azonenberg_pcb:EIA_0402_CAP_NOSILK, F.Cu at (302.7, 185.7)
- added C83: 0.47 uF, azonenberg_pcb:EIA_0402_CAP_NOSILK, F.Cu at (292.5, 196.0)
- added C84: 0.47 uF, azonenberg_pcb:EIA_0402_CAP_NOSILK, F.Cu at (302.7, 184.2)
- added C85: 0.47 uF, azonenberg_pcb:EIA_0402_CAP_NOSILK, F.Cu at (275.0, 198.6)
- added C86: 0.47 uF, azonenberg_pcb:EIA_0402_CAP_NOSILK, F.Cu at (273.2, 192.9)
- added C87: 0.47 uF, azonenberg_pcb:EIA_0402_CAP_NOSILK, F.Cu at (275.7, 192.9)
- added C88: 0.47 uF, azonenberg_pcb:EIA_0402_CAP_NOSILK, F.Cu at (270.0, 198.9)
- added C89: 0.47 uF, azonenberg_pcb:EIA_0402_CAP_NOSILK, F.Cu at (300.2, 181.2)
- added C9: 330 pF, azonenberg_pcb:EIA_0201_CAP_NOSILK, F.Cu at (30.0, 142.0)
- added C90: 0.47 uF, azonenberg_pcb:EIA_0402_CAP_NOSILK, F.Cu at (272.5, 198.9)
- added C91: 0.47 uF, azonenberg_pcb:EIA_0402_CAP_NOSILK, F.Cu at (281.9, 190.3)
- added C92: 0.47 uF, azonenberg_pcb:EIA_0402_CAP_NOSILK, F.Cu at (278.2, 193.6)
- added C93: 0.47 uF, azonenberg_pcb:EIA_0402_CAP_NOSILK, F.Cu at (278.2, 195.1)
- added C94: 0.47 uF, azonenberg_pcb:EIA_0402_CAP_NOSILK, F.Cu at (273.3, 197.1)
- added C95: 0.47 uF, azonenberg_pcb:EIA_0402_CAP_NOSILK, F.Cu at (303.5, 179.4)
- added C96: 0.47 uF, azonenberg_pcb:EIA_0402_CAP_NOSILK, F.Cu at (275.0, 200.1)
- added C97: 0.47 uF, azonenberg_pcb:EIA_0402_CAP_NOSILK, F.Cu at (281.9, 191.8)
- added C98: 0.47 uF, azonenberg_pcb:EIA_0402_CAP_NOSILK, F.Cu at (300.2, 182.7)
- added C99: 0.47 uF, azonenberg_pcb:EIA_0402_CAP_NOSILK, F.Cu at (275.8, 197.1)
- added F1: 3A, azonenberg_pcb:EIA_0603_RES_NOSILK, F.Cu at (290.5, 234.6)
- added FB1: MPZ2012S101AT000, azonenberg_pcb:EIA_0805_CAP_NOSILK, F.Cu at (292.5, 231.4)
- added FB2: BLM31KN121SZ1L, azonenberg_pcb:EIA_1206_CAP_NOSILK, F.Cu at (274.4, 187.2)
- added FB3: BLM31KN121SZ1L, azonenberg_pcb:EIA_1206_CAP_NOSILK, F.Cu at (274.4, 195.1)
- added FB4: BLM15PX121SN1D, azonenberg_pcb:EIA_0402_CAP_NOSILK, F.Cu at (280.7, 193.6)
- added FB5: BLM15PX121SN1D, azonenberg_pcb:EIA_0402_CAP_NOSILK, F.Cu at (330.6, 195.7)
- added FB6: BLM15PX121SN1D, azonenberg_pcb:EIA_0402_CAP_NOSILK, F.Cu at (333.9, 192.7)
- added FID1: FIDUCIAL, azonenberg_pcb:FIDUCIAL_1MM, F.Cu at (231.0, 41.0)
- added FID2: FIDUCIAL, azonenberg_pcb:FIDUCIAL_1MM, B.Cu at (232.0, 36.0)
- added FID3: FIDUCIAL, azonenberg_pcb:FIDUCIAL_1MM, F.Cu at (239.0, 45.0)
- added FID4: FIDUCIAL, azonenberg_pcb:FIDUCIAL_1MM, F.Cu at (235.0, 43.0)
- added FID5: FIDUCIAL, azonenberg_pcb:FIDUCIAL_1MM, B.Cu at (236.0, 37.0)
- added FID6: FIDUCIAL, azonenberg_pcb:FIDUCIAL_1MM, B.Cu at (242.0, 39.0)
- added J1: SMA, azonenberg_pcb:CONN_SMA_EDGE_SAMTEC_SMA_J_P_H_ST_EM1, F.Cu at (14.9, 176.0)
- added J10: XILINX_JTAG, azonenberg_pcb:XILINX_JTAG_PTH_MOLEX_0878311420, F.Cu at (228.3, 182.3)
- added J11: SMA, azonenberg_pcb:CONN_SMA_EDGE_SAMTEC_SMA_J_P_H_ST_EM1, F.Cu at (280.3, 238.2)
- added J12: SMA, azonenberg_pcb:CONN_SMA_EDGE_SAMTEC_SMA_J_P_H_ST_EM1, F.Cu at (273.0, 244.3)
- added J13: SMA, azonenberg_pcb:CONN_SMA_EDGE_SAMTEC_SMA_J_P_H_ST_EM1, F.Cu at (320.4, 195.7)
- added J14: SMA, azonenberg_pcb:CONN_SMA_EDGE_SAMTEC_SMA_J_P_H_ST_EM1, F.Cu at (330.7, 183.8)
- added J15: SMA, azonenberg_pcb:CONN_SMA_EDGE_SAMTEC_SMA_J_P_H_ST_EM1, F.Cu at (312.1, 211.4)
- added J16: SMA, azonenberg_pcb:CONN_SMA_EDGE_SAMTEC_SMA_J_P_H_ST_EM1, F.Cu at (312.1, 205.5)
- added J17: SMA, azonenberg_pcb:CONN_SMA_EDGE_SAMTEC_SMA_J_P_H_ST_EM1, F.Cu at (269.5, 209.1)
- added J18: SMA, azonenberg_pcb:CONN_SMA_EDGE_SAMTEC_SMA_J_P_H_ST_EM1, F.Cu at (269.5, 215.0)
- added J19: JUMPER, azonenberg_pcb:CONN_HEADER_2.54MM_1x2, F.Cu at (223.2, 196.9)
- added J2: BARREL, azonenberg_pcb:CONN_CUI_PJ-058BH_HIPWR_BARREL_NOSLOT, F.Cu at (33.0, 270.0)
- added J20: JUMPER, azonenberg_pcb:CONN_HEADER_2.54MM_1x2, F.Cu at (241.5, 181.2)
- added J21: JUMPER, azonenberg_pcb:CONN_HEADER_2.54MM_1x2, F.Cu at (249.1, 193.4)
- added J22: SMA, azonenberg_pcb:CONN_SMA_EDGE_SAMTEC_SMA_J_P_H_ST_EM1, F.Cu at (322.7, 189.8)
- added J23: SMA, azonenberg_pcb:CONN_SMA_EDGE_SAMTEC_SMA_J_P_H_ST_EM1, F.Cu at (322.7, 183.8)
- added J24: SMA, azonenberg_pcb:CONN_SMA_EDGE_SAMTEC_SMA_J_P_H_ST_EM1, F.Cu at (240.1, 191.1)
- added J25: SMA, azonenberg_pcb:CONN_SMA_EDGE_SAMTEC_SMA_J_P_H_ST_EM1, F.Cu at (231.3, 199.5)
- added J26: PMOD_HOST, azonenberg_pcb:CONN_HEADER_2.54MM_2x6_RA_PMOD_HOST, F.Cu at (227.7, 189.2)
- added J3: SMA, azonenberg_pcb:CONN_SMA_EDGE_SAMTEC_SMA_J_P_H_ST_EM1, F.Cu at (15.9, 138.0)
- added J4: SMA, azonenberg_pcb:CONN_SMA_EDGE_SAMTEC_SMA_J_P_H_ST_EM1, F.Cu at (15.9, 151.0)
- added J5: SMA, azonenberg_pcb:CONN_SMA_EDGE_SAMTEC_SMA_J_P_H_ST_EM1, F.Cu at (15.9, 125.0)
- added J6: XILINX_JTAG, azonenberg_pcb:XILINX_JTAG_PTH_MOLEX_0878311420, F.Cu at (274.6, 182.3)
- added J7: CONN_INTEGRALSTICK_FPGA_HOST, azonenberg_pcb:CONN_SAMTEC_QSH-060-01-L-D-A, F.Cu at (61.0, 78.0)
- added J8: CONN_INTEGRALSTICK_MCU_HOST, azonenberg_pcb:CONN_SAMTEC_QSH-060-01-L-D-A, F.Cu at (134.0, 78.0)
- added J9: 0826-1G1T-23-F, azonenberg_pcb:CONN_BELFUSE_0826_1G1T_23_F, F.Cu at (192.0, 99.0)
- added JP1: JUMPER_0402, azonenberg_pcb:EIA_0402_JUMPER, F.Cu at (38.8, 129.8)
- added JP2: JUMPER_0402, azonenberg_pcb:EIA_0402_JUMPER, F.Cu at (324.0, 201.1)
- added JP3: JUMPER_0402, azonenberg_pcb:EIA_0402_JUMPER, F.Cu at (327.5, 201.1)
- added JP4: JUMPER_0402, azonenberg_pcb:EIA_0402_JUMPER, F.Cu at (285.5, 209.4)
- added JP5: JUMPER_0402, azonenberg_pcb:EIA_0402_JUMPER, F.Cu at (278.2, 216.9)
- added JP6: JUMPER_0402, azonenberg_pcb:EIA_0402_JUMPER, F.Cu at (273.4, 221.7)
- added JP8: JUMPER_0402, azonenberg_pcb:EIA_0402_JUMPER, F.Cu at (326.1, 223.4)
- added M1: TRACEPAD, azonenberg_pcb:SERIALNUM_MOLEX_0916580020, F.Cu at (279.0, 245.7)
- added M2: LOGO1, azonenberg_pcb:LONGTHING-1200DPI, F.Cu at (228.0, 49.0)
- added M3: LOGO2, w_logo:Logo_silk_OSHW_6x6mm, F.Cu at (261.0, 50.0)
- added M4: LOGO3, w_logo:Logo_silk_polarity_center_5x1.4mm, F.Cu at (243.0, 50.0)
- added M5: LOGO4, w_logo:Logo_silk_ROHS_5x2.8mm, F.Cu at (249.0, 50.0)
- added M6: LOGO5, w_logo:Logo_silk_warning_5x4.2mm, F.Cu at (237.0, 50.0)
- added M7: LOGO6, w_logo:Logo_silk_WEEE_3.4x5mm, F.Cu at (255.0, 50.0)
- added Q1: SSM6N58NU, azonenberg_pcb:DFN_6_0.65MM_2x2MM_GDS, F.Cu at (252.4, 197.8)
- added R1: PS3216GT2-R50-T1‎, azonenberg_pcb:SPLITTER_SUSUMU_PS3216G, F.Cu at (27.8, 176.0)
- added R10: 100, azonenberg_pcb:EIA_0402_RES_NOSILK, F.Cu at (285.0, 199.0)
- added R100: DNP, azonenberg_pcb:EIA_0402_RES_NOSILK, F.Cu at (292.5, 197.5)
- added R101: DNP, azonenberg_pcb:EIA_0402_RES_NOSILK, F.Cu at (300.2, 188.7)
- added R102: 10K, azonenberg_pcb:EIA_0402_RES_NOSILK, F.Cu at (290.0, 199.0)
- added R103: 10K, azonenberg_pcb:EIA_0402_RES_NOSILK, F.Cu at (282.5, 198.1)
- added R104: 10K, azonenberg_pcb:EIA_0402_RES_NOSILK, F.Cu at (307.7, 236.2)
- added R105: 10K, azonenberg_pcb:EIA_0402_RES_NOSILK, F.Cu at (316.0, 228.2)
- added R106: 5K 0.1%, azonenberg_pcb:EIA_0402_RES_NOSILK, F.Cu at (294.5, 275.1)
- added R107: 5K 0.1%, azonenberg_pcb:EIA_0402_RES_NOSILK, F.Cu at (290.0, 280.4)
- added R108: 5K 0.1%, azonenberg_pcb:EIA_0402_RES_NOSILK, F.Cu at (294.5, 276.6)
- added R109: 20K 0.1%, azonenberg_pcb:EIA_0402_RES_NOSILK, F.Cu at (293.2, 278.1)
- added R11: 1K, azonenberg_pcb:EIA_0402_RES_NOSILK, F.Cu at (302.7, 181.2)
- added R110: 20K 0.1%, azonenberg_pcb:EIA_0402_RES_NOSILK, F.Cu at (292.5, 280.4)
- added R111: 20K 0.1%, azonenberg_pcb:EIA_0402_RES_NOSILK, F.Cu at (290.7, 278.9)
- added R112: 953, azonenberg_pcb:EIA_0402_RES_NOSILK, F.Cu at (252.5, 240.9)
- added R113: 953, azonenberg_pcb:EIA_0402_RES_NOSILK, F.Cu at (240.1, 253.4)
- added R114: 453, azonenberg_pcb:EIA_0402_RES_NOSILK, F.Cu at (228.7, 264.9)
- added R115: 453, azonenberg_pcb:EIA_0402_RES_NOSILK, F.Cu at (240.1, 251.9)
- added R116: 453, azonenberg_pcb:EIA_0402_RES_NOSILK, F.Cu at (226.2, 266.4)
- added R117: 453, azonenberg_pcb:EIA_0402_RES_NOSILK, F.Cu at (244.0, 247.7)
- added R118: 453, azonenberg_pcb:EIA_0402_RES_NOSILK, F.Cu at (232.6, 253.0)
- added R119: 453, azonenberg_pcb:EIA_0402_RES_NOSILK, F.Cu at (228.7, 263.4)
- added R12: 33, azonenberg_pcb:EIA_0402_RES_NOSILK, F.Cu at (287.5, 196.0)
- added R120: 453, azonenberg_pcb:EIA_0402_RES_NOSILK, F.Cu at (252.5, 239.4)
- added R121: 453, azonenberg_pcb:EIA_0402_RES_NOSILK, F.Cu at (233.5, 259.0)
- added R122: 453, azonenberg_pcb:EIA_0402_RES_NOSILK, F.Cu at (246.4, 246.2)
- added R123: 453, azonenberg_pcb:EIA_0402_RES_NOSILK, F.Cu at (231.0, 260.9)
- added R124: 453, azonenberg_pcb:EIA_0402_RES_NOSILK, F.Cu at (235.7, 256.0)
- added R125: 453, azonenberg_pcb:EIA_0402_RES_NOSILK, F.Cu at (249.2, 242.0)
- added R126: 453, azonenberg_pcb:EIA_0402_RES_NOSILK, F.Cu at (241.5, 250.4)
- added R127: 453, azonenberg_pcb:EIA_0402_RES_NOSILK, F.Cu at (244.0, 249.2)
- added R128: 10K, azonenberg_pcb:EIA_0402_RES_NOSILK, F.Cu at (323.5, 207.3)
- added R129: 10K, azonenberg_pcb:EIA_0402_RES_NOSILK, F.Cu at (323.5, 205.8)
- added R13: DNP, azonenberg_pcb:EIA_0402_RES_NOSILK, F.Cu at (287.5, 194.5)
- added R130: 10K, azonenberg_pcb:EIA_0402_RES_NOSILK, F.Cu at (295.5, 207.6)
- added R131: 909, azonenberg_pcb:EIA_0402_RES_NOSILK, F.Cu at (292.5, 212.4)
- added R132: 909, azonenberg_pcb:EIA_0402_RES_NOSILK, F.Cu at (293.3, 210.9)
- added R133: 909, azonenberg_pcb:EIA_0402_RES_NOSILK, F.Cu at (286.2, 217.2)
- added R134: 909, azonenberg_pcb:EIA_0402_RES_NOSILK, F.Cu at (283.9, 220.1)
- added R135: 909, azonenberg_pcb:EIA_0402_RES_NOSILK, F.Cu at (298.0, 206.1)
- added R136: 909, azonenberg_pcb:EIA_0402_RES_NOSILK, F.Cu at (288.7, 215.7)
- added R137: 10K, azonenberg_pcb:EIA_0402_RES_NOSILK, F.Cu at (294.5, 273.6)
- added R14: 150, azonenberg_pcb:EIA_0402_RES_NOSILK, F.Cu at (325.6, 196.4)
- added R15: 1K 1%, azonenberg_pcb:EIA_0402_RES_NOSILK, F.Cu at (334.6, 187.1)
- added R16: 470, azonenberg_pcb:EIA_0402_RES_NOSILK, F.Cu at (220.4, 204.6)
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Routing:
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- added copper zone on F.Cu, net /GND
Other:
- net class Default: via_dia 0.55 -> 0.5; via_drill 0.3 -> 0.2
- board text added: "1"
- board text added: "2"
- board text added: "3"
- board text added: "4"
- board text added: "5"
- board text added: "6"
- board text added: "7"
- board text added: "8"
- board text added: "CLKIN"
- board text added: "CLKIN+"
- board text added: "CLKIN-"
- board text added: "EXT REFCLK"
- board text added: "M"
- board text added: "S"

Commit message: Began layout on clock recovery block
Parts:
- C60: moved to B.Cu
- moved C63 256.7 mm to (45.6, 133.4), turned to 180 degrees
- moved C62 256.2 mm to (51.5, 126.5), turned to 180 degrees
- moved C64 254.9 mm to (45.6, 133.9), turned to 180 degrees
- moved C61 252.5 mm to (51.5, 126.0), turned to 180 degrees
- moved C58 237.1 mm to (52.3, 125.1)
- moved C60 231.7 mm to (50.2, 121.7), turned to 90 degrees
- moved U13 34.8 mm to (52.0, 123.1)
- moved U5 31.2 mm to (60.8, 128.2), turned to 270 degrees
- moved U6 30.5 mm to (48.4, 125.0)
- moved C65 0.74 mm to (297.0, 194.6)
Connections:
- U3 pad 4: /CDR/CDR_EXTCLK_N -> /PLL/EXTCLK_N
- U3 pad 5: /CDR/CDR_EXTCLK_P -> /PLL/EXTCLK_P
- U3 pad 7: /PLL/EXTCLK_N -> /CDR/CDR_EXTCLK_N
- U3 pad 8: /PLL/EXTCLK_P -> /CDR/CDR_EXTCLK_P
- U6 pad 4: /CDR/SERDES_REFCLK0_P -> /CDR/SERDES_REFCLK0_N
- U6 pad 5: /CDR/SERDES_REFCLK0_N -> /CDR/SERDES_REFCLK0_P
Routing:
- net /GND: track 246.3 -> 358.5 mm, vias 150 -> 229
- net /3V3_PLL: track 0.00 -> 28.5 mm, vias 0 -> 2
- net /CDR/SRC1_AC_P: track 0.00 -> 12.7 mm, vias 0 -> 2
- net /CDR/SRC1_AC_N: track 0.00 -> 12.7 mm, vias 0 -> 2
- net /CDR/SRC0_AC_N: track 0.00 -> 9.03 mm
- net /CDR/SRC0_AC_P: track 0.00 -> 9.03 mm
- net /OSC_OE: track 0.00 -> 8.06 mm, vias 0 -> 1
- net /OSC_PWR_EN: track 0.00 -> 7.95 mm, vias 0 -> 1
- net /CDR/CDR_EXTCLK_N: track 8.21 -> 4.78 mm
- net /CDR/CDR_EXTCLK_P: track 7.91 -> 4.76 mm
- net /CDR/SERDES_REFCLK0_P: track 0.00 -> 2.10 mm
- net /CDR/SERDES_REFCLK0_N: track 0.00 -> 1.98 mm
- net /CDR/OSC_VDD: track 0.00 -> 1.57 mm, vias 0 -> 1
- net /CDR/SCLKO_DC_P: vias 0 -> 1
- net /CDR/SCLKO_DC_N: vias 0 -> 1

Commit message: Finished initial layout of CDR subsystem
Parts:
- C100, C101, C102, C56, C57, C59, C65, C66, C67, C68, C69, C70, C71, C72, C73, C74, C75, C76, C77, C78, C79, C80, C81, C82, C83, C84, C85, C86, C87, C88, C89, C90, C91, C92, C93, C94, C95, C96, C97, C98, C99, FB2, FB3, FB4, R10, R100, R101, R102, R103, R11, R12, R13, R2, R23, R3, R4, R5, R6, R7, R74, R75, R8, R9, R97, R98, R99: moved to B.Cu
- moved R11 253.4 mm to (54.5, 130.0), turned to 90 degrees
- moved R5 253.1 mm to (56.8, 122.8)
- moved R101 252.1 mm to (54.2, 133.2), turned to 90 degrees
- moved C71 251.4 mm to (53.1, 134.9), turned to 90 degrees
- moved R6 251.3 mm to (55.8, 125.8)
- moved C84 249.9 mm to (59.8, 125.8), turned to 180 degrees
- moved R102 249.6 mm to (52.8, 121.6)
- moved C82 249.4 mm to (61.2, 123.2), turned to 90 degrees
- moved R103 247.1 mm to (47.0, 123.2)
- moved C95 247.1 mm to (62.8, 123.8), turned to 180 degrees
- moved C79 246.6 mm to (60.2, 130.2), turned to 270 degrees
- moved R2 246.6 mm to (59.2, 133.2), turned to 90 degrees
- moved C98 246.3 mm to (60.2, 127.2), turned to 90 degrees
- moved R4 245.2 mm to (55.8, 123.8), turned to 180 degrees
- moved C89 244.9 mm to (60.2, 132.2), turned to 270 degrees
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Routing:
- net /GND: track 358.5 -> 430.2 mm, vias 229 -> 290
- net /1V8: track 44.0 -> 91.1 mm, vias 12 -> 23
- net /1V0: track 0.00 -> 43.8 mm, vias 0 -> 19
- net /CDR/A1V8_PLL_SERDES: track 0.00 -> 29.9 mm, vias 0 -> 6
- net /CDR/A1V0_SERDES: track 0.00 -> 21.8 mm, vias 0 -> 8
- net /SERDES_MODE_SEL: track 0.00 -> 14.5 mm, vias 0 -> 1
- net /SERDES_MDC: track 0.00 -> 14.4 mm, vias 0 -> 1
- net /OSC_FS0: track 0.00 -> 13.7 mm, vias 0 -> 1
- net /CDR/A1V0T_SERDES: track 0.00 -> 13.5 mm, vias 0 -> 5
- net /CDR/SERDES_TCK: track 0.00 -> 13.1 mm, vias 0 -> 1
- net /CDR/SERDES_TMS: track 0.00 -> 12.4 mm, vias 0 -> 1
- net /CDR/SERDES_TDI: track 0.00 -> 12.2 mm, vias 0 -> 1
- net /SERDES_POWER_EN: track 0.00 -> 11.8 mm, vias 0 -> 1
- net /SERDES_MDIO: track 0.00 -> 11.6 mm, vias 0 -> 2
- net /OSC_OS: track 0.00 -> 11.0 mm, vias 0 -> 1
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Other:
- board text added: "CLOCK RECOVERY"

Commit message: Moved CDR block down so it's closer to the level trigger
Parts:
- moved M5 119.0 mm to (146.0, 62.8)
- moved U14 20.1 mm to (50.8, 127.0)
- moved U15 20.1 mm to (64.8, 127.0)
- moved C61 16.0 mm to (51.5, 142.1)
- moved C62 16.0 mm to (51.5, 142.6)
- moved C67 16.0 mm to (67.6, 139.8)
- moved FB2 16.0 mm to (66.0, 137.3)
- moved R98 16.0 mm to (57.2, 137.8)
- moved C100 16.0 mm to (56.8, 140.8)
- moved C101 16.0 mm to (61.2, 143.2)
- moved C102 16.0 mm to (61.2, 145.2)
- moved C56 16.0 mm to (65.5, 151.4)
- moved C57 16.0 mm to (66.0, 151.4)
- moved C58 16.0 mm to (52.3, 141.1)
- moved C59 16.0 mm to (49.0, 140.2)
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Connections:
- U3 pad 4: /PLL/EXTCLK_N -> /CDR/CDR_EXTCLK_N
- U3 pad 5: /PLL/EXTCLK_P -> /CDR/CDR_EXTCLK_P
- U3 pad 7: /CDR/CDR_EXTCLK_N -> /PLL/EXTCLK_N
- U3 pad 8: /CDR/CDR_EXTCLK_P -> /PLL/EXTCLK_P
Routing:
- net /CDR/CDR_EXTCLK_P: track 4.76 -> 14.2 mm
- net /CDR/CDR_EXTCLK_N: track 4.78 -> 14.2 mm
- net /PLL/EXTCLK_N: track 7.55 -> 0.79 mm
- net /PLL/EXTCLK_P: track 7.25 -> 0.94 mm
- net /SERDES_MDC: track 14.4 -> 12.4 mm
- net /GND: track 430.2 -> 431.5 mm, vias 290 -> 289
- net /CDR/SRC1_AC_P: track 12.7 -> 11.9 mm
- net /CDR/SRC1_AC_N: track 12.7 -> 11.9 mm
