File: boards/freesample/freesample.sch (KiCad schematic (older format))
At the start: 20 parts, among them J1 SMA, J11 SMA, J12 SMA, J2 BARREL, M1 TRACEPAD, M2 LOGO1, M3 LOGO2, M4 LOGO3, M5 LOGO4, M6 LOGO5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

Commit message: Tweaks to PLL and CDR layout, swapped a few signals around. Began work on level trigger and ADC layout.
Connections:
- net VIN_0 renamed ADC_DIN
- net VIN_1 renamed LTRIG_DIN
Other:
- moved on the sheet: J1, R1
Changed lines of the file:
@@
 L freesample-rescue:CONN_COAXIAL-conn J1
 U 1 1 5C201EC1
-P 750 850
-F 0 "J1" H 703 1088 50  0000 C CNN
-F 1 "SMA" H 703 997 50  0000 C CNN
-F 2 "azonenberg_pcb:CONN_SMA_EDGE_SAMTEC_SMA_J_P_H_ST_EM1" H 750 850 50  0001 C CNN
-F 3 "" H 750 850 50  0001 C CNN
-	1    750  850
+P 650 850
+F 0 "J1" H 603 1088 50  0000 C CNN
+F 1 "SMA" H 603 997 50  0000 C CNN
+F 2 "azonenberg_pcb:CONN_SMA_EDGE_SAMTEC_SMA_J_P_H_ST_EM1" H 650 850 50  0001 C CNN
+F 3 "" H 650 850 50  0001 C CNN
+	1    650  850
 	-1   0    0    -1
 $EndComp
-Text Label 750  1200 0    50   ~ 10
-GND
-Wire Wire Line
-	750  1200 750  1050
-Text Label 900  850  0    50   ~ 10
+Text Label 650  1200 0    50   ~ 0
+GND
+Wire Wire Line
+	650  1200 650  1050
+Text Label 800  850  0    50   ~ 0
 VIN
 $Comp
 L analog-azonenberg:SPLITTER_SUSUMU_PS R1
 U 1 1 5C20338C
-P 1350 1000
-F 0 "R1" H 1600 1375 50  0000 C CNN
-F 1 "PS3216GT2-R50-T1‎" H 1600 1284 50  0000 C CNN
-F 2 "azonenberg_pcb:SPLITTER_SUSUMU_PS3216G" H 1350 1000 50  0001 C CNN
-F 3 "" H 1350 1000 50  0001 C CNN
-	1    1350 1000
+P 1250 1000
+F 0 "R1" H 1500 1375 50  0000 C CNN
+F 1 "PS3216GT2-R50-T1‎" H 1500 1284 50  0000 C CNN
+F 2 "azonenberg_pcb:SPLITTER_SUSUMU_PS3216G" H 1250 1000 50  0001 C CNN
+F 3 "" H 1250 1000 50  0001 C CNN
+	1    1250 1000
 	1    0    0    -1
 $EndComp
 Wire Wire Line
-	1250 850  900  850
+	1150 850  800  850
 $Sheet
 S 2750 1800 1100 800
@@
 Wire Wire Line
 	5550 1450 5650 1450
-Wire Wire Line
-	1950 850  2750 850
-Text Label 2650 1250 2    50   ~ 10
+Text Label 2650 1250 2    50   ~ 0
 3V3
 Wire Wire Line
 	2650 1250 2750 1250
-Text Label 2650 1350 2    50   ~ 10
+Text Label 2650 1350 2    50   ~ 0
 1V8
-Text Label 2650 1450 2    50   ~ 10
-GND
-Text Label 2650 1550 2    50   ~ 10
+Text Label 2650 1450 2    50   ~ 0
+GND
+Text Label 2650 1550 2    50   ~ 0
 3V0_N
 Wire Wire Line
@@
 Wire Wire Line
 	2650 1350 2750 1350
-Text Label 2050 850  0    50   ~ 10
-VIN_0
-Text Label 2050 950  0    50   ~ 10
-VIN_1
-Wire Wire Line
-	1950 950  2050 950
-Wire Wire Line
-	2050 950  2050 1900
-Wire Wire Line
-	2050 1900 2750 1900
+Text Label 1850 850  0    50   ~ 0
+ADC_DIN
+Text Label 1850 950  0    50   ~ 0
+LTRIG_DIN
 Text Label 2650 2200 2    50   ~ 10
 3V3
@@
 Wire Wire Line
 	2750 2500 2650 2500
-Text Label 2650 950  2    50   ~ 10
+Text Label 2650 950  2    50   ~ 0
 LTRIG_VT
-Text Label 2650 2000 2    50   ~ 10
+Text Label 2650 2000 2    50   ~ 0
 ADC_VT
 Wire Wire Line
@@
 Wire Wire Line
 	4650 3250 10450 3250
-Text Label 10400 1100 2    50   ~ 10
+Text Label 10400 1100 2    50   ~ 0
 SAMP_MUXSEL0
 Wire Wire Line
 	10400 1100 10450 1100
-Text Label 10400 1200 2    50   ~ 10
+Text Label 10400 1200 2    50   ~ 0
 SAMP_MUXSEL1
 Wire Wire Line
@@
 Wire Wire Line
 	13000 4500 9450 4500
-Text Label 10400 1400 2    50   ~ 10
+Text Label 10400 1400 2    50   ~ 0
 3V3_CLKBUF
 Wire Wire Line
 	10400 1400 10450 1400
-Text Label 10400 1500 2    50   ~ 10
+Text Label 10400 1500 2    50   ~ 0
 GND
 Wire Wire Line
@@
 	750  2200 850  2200
 NoConn ~ 13100 1000
-Text Label 13200 900  0    50   ~ 10
+Text Label 13200 900  0    50   ~ 0
 GND
 Wire Wire Line
 	13200 900  13100 900
-Text Label 13200 800  0    50   ~ 10
+Text Label 13200 800  0    50   ~ 0
 12V0_RAW
 Wire Wire Line
@@
 	0    1    1    0
 $EndComp
-Text Label 14800 800  0    50   ~ 10
+Text Label 14800 800  0    50   ~ 0
 12V0
 Text Label 6800 5000 0    50   ~ 10
@@
 Wire Wire Line
 	5550 2450 5650 2450
-Text Label 2650 1150 2    50   ~ 10
+Text Label 2650 1150 2    50   ~ 0
 3V3_CLKBUF
 Wire Wire Line
@@
 Wire Wire Line
 	5550 1650 5650 1650
-Text Notes 600  1350 0    50   ~ 10
+Text Notes 600  1350 0    50   ~ 0
 MAX -2V to +2V INPUT
 Text Label 9800 2300 0    50   ~ 0
@@
 	-1   0    0    1
 $EndComp
-Text Label 1250 950  2    50   ~ 10
+Text Label 1150 950  2    50   ~ 0
 GND
 Text Label 4750 4900 2    50   ~ 10
@@
 	-1   0    0    1
 $EndComp
+Text Label 2650 1900 2    50   ~ 0
+ADC_DIN
+Wire Wire Line
+	2650 1900 2750 1900
+Text Label 2650 850  2    50   ~ 0
+LTRIG_DIN
+Wire Wire Line
+	2650 850  2750 850
 $EndSCHEMATC

Commit message: Finished initial layout of level trigger and ADC subsystems
Changed lines of the file:
@@
 Text Label 1850 950  0    50   ~ 0
 LTRIG_DIN
-Text Label 2650 2200 2    50   ~ 10
+Text Label 2650 2200 2    50   ~ 0
 3V3
-Text Label 2650 2400 2    50   ~ 10
+Text Label 2650 2400 2    50   ~ 0
 GND
-Text Label 2650 2500 2    50   ~ 10
+Text Label 2650 2500 2    50   ~ 0
 3V0_N
-Text Label 2650 2300 2    50   ~ 10
+Text Label 2650 2300 2    50   ~ 0
 1V8
 Wire Wire Line
@@
 Wire Wire Line
 	8300 1200 8400 1200
-Text Label 4000 1900 0    50   ~ 10
+Text Label 4000 1900 0    50   ~ 0
 ADC_OUT_P
 Wire Wire Line
 	4000 1900 3850 1900
-Text Label 4000 2000 0    50   ~ 10
+Text Label 4000 2000 0    50   ~ 0
 ADC_OUT_N
 Wire Wire Line

Commit message: Initial layout of coarse delay line
Changed lines of the file:
@@
 Sheet 1 12
 Title "FREESAMPLE Oscilloscope"
-Date "2019-03-23"
+Date "2019-03-25"
 Rev "0.1"
 Comp "Andrew D. Zonenberg / Antikernel Labs"
@@
 Wire Wire Line
 	10400 1500 10450 1500
-Text Label 7850 4700 2    50   ~ 10
+Text Label 7850 4700 2    50   ~ 0
 3V3
 Wire Wire Line
 	7850 4700 7950 4700
-Text Label 7850 4800 2    50   ~ 10
+Text Label 7850 4800 2    50   ~ 0
 GND
 Wire Wire Line
 	7850 4800 7950 4800
-Text Label 7850 4900 2    50   ~ 10
+Text Label 7850 4900 2    50   ~ 0
 3V3_N
 Wire Wire Line
 	7850 4900 7950 4900
-Text Label 7850 5300 2    50   ~ 10
+Text Label 7850 5300 2    50   ~ 0
 COARSE_EN
 Wire Wire Line
 	7850 5300 7950 5300
-Text Label 7850 5400 2    50   ~ 10
+Text Label 7850 5400 2    50   ~ 0
 COARSE_SLOAD
 Wire Wire Line
 	7850 5400 7950 5400
-Text Label 7850 5500 2    50   ~ 10
+Text Label 7850 5500 2    50   ~ 0
 COARSE_SDIN
 Wire Wire Line
 	7850 5500 7950 5500
-Text Label 7850 5600 2    50   ~ 10
+Text Label 7850 5600 2    50   ~ 0
 COARSE_SCLK
 Wire Wire Line
 	7850 5600 7950 5600
-Text Label 7850 5800 2    50   ~ 10
+Text Label 7850 5800 2    50   ~ 0
 FINE_SEL0_P
 Wire Wire Line
 	7850 5800 7950 5800
-Text Label 7850 5900 2    50   ~ 10
+Text Label 7850 5900 2    50   ~ 0
 FINE_SEL0_N
 Wire Wire Line
 	7850 5900 7950 5900
-Text Label 7850 6100 2    50   ~ 10
+Text Label 7850 6100 2    50   ~ 0
 FINE_SEL1_P
 Wire Wire Line
 	7850 6100 7950 6100
-Text Label 7850 6200 2    50   ~ 10
+Text Label 7850 6200 2    50   ~ 0
 FINE_SEL1_N
 Wire Wire Line
 	7850 6200 7950 6200
-Text Label 7850 6400 2    50   ~ 10
+Text Label 7850 6400 2    50   ~ 0
 FINE_SEL2_P
 Wire Wire Line
 	7850 6400 7950 6400
-Text Label 7850 6500 2    50   ~ 10
+Text Label 7850 6500 2    50   ~ 0
 FINE_SEL2_N
 Wire Wire Line
 	7850 6500 7950 6500
-Text Label 7850 6700 2    50   ~ 10
+Text Label 7850 6700 2    50   ~ 0
 FINE_SEL3_P
 Wire Wire Line
 	7850 6700 7950 6700
-Text Label 7850 6800 2    50   ~ 10
+Text Label 7850 6800 2    50   ~ 0
 FINE_SEL3_N
 Wire Wire Line
 	7850 6800 7950 6800
-Text Label 7850 7000 2    50   ~ 10
+Text Label 7850 7000 2    50   ~ 0
 FINE_SEL4_P
 Wire Wire Line
 	7850 7000 7950 7000
-Text Label 7850 7100 2    50   ~ 10
+Text Label 7850 7100 2    50   ~ 0
 FINE_SEL4_N
 Wire Wire Line

Commit message: Initial layout work on one-shot. Nowhere near done.
Changed lines of the file:
@@
 Sheet 1 12
 Title "FREESAMPLE Oscilloscope"
-Date "2019-03-28"
+Date "2019-03-31"
 Rev "0.1"
 Comp "Andrew D. Zonenberg / Antikernel Labs"
@@
 Wire Wire Line
 	7300 2950 10450 2950
-Text Label 4750 4100 2    50   ~ 10
+Text Label 4750 4100 2    50   ~ 0
 ONESHOT_RST_P
-Text Label 4750 4200 2    50   ~ 10
+Text Label 4750 4200 2    50   ~ 0
 ONESHOT_RST_N
 Wire Wire Line
 	4850 4200 4750 4200
-Text Label 6800 4700 0    50   ~ 10
+Text Label 6800 4700 0    50   ~ 0
 TRIGGERED_P
 Wire Wire Line
 	6800 4700 6650 4700
-Text Label 6800 4800 0    50   ~ 10
+Text Label 6800 4800 0    50   ~ 0
 TRIGGERED_N
 Wire Wire Line
@@
 Text Label 14800 800  0    50   ~ 0
 12V0
-Text Label 6800 5000 0    50   ~ 10
+Text Label 6800 5000 0    50   ~ 0
 RANGE_SEL
 Wire Wire Line
@@
 Wire Wire Line
 	4750 4900 4850 4900
-Text Label 4750 5000 2    50   ~ 10
-GND
-Text Label 4750 4800 2    50   ~ 10
+Text Label 4750 5000 2    50   ~ 0
+GND
+Text Label 4750 4800 2    50   ~ 0
 2V5
 Wire Wire Line
@@
 Text Label 1950 10450 0    50   ~ 10
 SERDES_POWER_EN
-Text Label 4750 4700 2    50   ~ 10
+Text Label 4750 4700 2    50   ~ 0
 3V3_CLKBUF
 Wire Wire Line
@@
 Wire Wire Line
 	4850 5350 4250 5350
-Text Label 4100 5000 2    50   ~ 10
-GND
-Text Label 4100 5550 2    50   ~ 10
+Text Label 4100 5000 2    50   ~ 0
+GND
+Text Label 4100 5550 2    50   ~ 0
 GND
 Wire Wire Line
 	4250 5200 4850 5200
-Text Notes 4100 5750 0    50   ~ 10
+Text Notes 4100 5750 0    50   ~ 0
 Phase shifted sampling clock out\nfor debugging or external logic
 $Comp
@@
 Text Label 1150 950  2    50   ~ 0
 GND
-Text Label 4750 4900 2    50   ~ 10
+Text Label 4750 4900 2    50   ~ 0
 1V8
 Wire Wire Line
